File: pcb/revisions/rev-1.0__or/dormin_v1.kicad_pcb (KiCad board)
At the start: 2 copper layers, 156.2 x 118.2 mm, 68 parts, among them SW1 SW_PUSH-MX_CHOC, SW10 SW_PUSH-MX_CHOC, SW11 SW_PUSH-MX_CHOC, SW12 SW_PUSH-MX_CHOC, SW13 SW_PUSH-MX_CHOC, SW14 SW_PUSH-MX_CHOC, SW15 SW_PUSH-MX_CHOC, SW16 SW_PUSH-MX_CHOC, SW17 SW_PUSH-MX_CHOC, SW19 SW_PUSH-MX_CHOC, SW2 SW_PUSH-MX_CHOC, SW20 SW_PUSH-MX_CHOC, SW21 SW_PUSH-MX_CHOC, SW22 SW_PUSH-MX_CHOC, SW3 SW_PUSH-MX_CHOC, SW4 SW_PUSH-MX_CHOC, SW5 SW_PUSH-MX_CHOC, SW6 SW_PUSH-MX_CHOC, SW7 SW_PUSH-MX_CHOC, SW8 SW_PUSH-MX_CHOC, SW9 SW_PUSH-MX_CHOC, U1 Seeeduino Xiao nRF52840

Commit message: refactor: added initial versions of the pcb
Connections:
- U1 pad 11: col4 -> LED
- U1 pad 18: LED -> col4
- U1 pad 20: unconnected-(U1-CLK-Pad20) -> Net-(U1-CLK)
Changed lines of the file:
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@@
 			(layers "*.Cu" "*.Mask")
 			(remove_unused_layers no)
-			(net "col4")
+			(net "LED")
 			(pinfunction "P1.15_11")
 			(pintype "bidirectional")
@@
 			(layers "F.Cu" "F.Mask")
 			(roundrect_rratio 0.25)
-			(net "col4")
+			(net "LED")
 			(pinfunction "P1.15_11")
 			(pintype "bidirectional")
@@
 			(remove_unused_layers no)
 			(roundrect_rratio 0.25)
-			(net "LED")
+			(net "col4")
 			(pinfunction "P0.10_18")
 			(pintype "bidirectional")
@@
 			(layers "F.Cu" "F.Mask")
 			(roundrect_rratio 0.25)
-			(net "LED")
+			(net "col4")
 			(pinfunction "P0.10_18")
 			(pintype "bidirectional")
@@
 			(layers "*.Cu" "*.Mask")
 			(remove_unused_layers no)
-			(net "unconnected-(U1-CLK-Pad20)")
+			(net "Net-(U1-CLK)")
 			(pinfunction "CLK_20")
 			(pintype "bidirectional")
