File: keyboard/kicad/revisions/dormin-rev_1.0/dormin-rev_1.0.kicad_sch (KiCad schematic)
At the start: 67 parts, among them SW1 SW_Push, SW10 SW_Push, SW11 SW_Push, SW12 SW_Push, SW13 SW_Push, SW14 SW_Push, SW15 SW_Push, SW16 SW_Push, SW17 SW_Push, SW18 SW_Push, SW19 SW_Push, SW2 SW_Push, SW20 SW_Push, SW21 SW_Push, SW3 SW_Push, SW4 SW_Push, SW5 SW_Push, SW6 SW_Push, SW7 SW_Push, SW8 SW_Push, SW9 SW_Push, U1 Seeeduino Xiao nRF52840

Commit message: feat: update ergogen and kicad
Parts:
- removed JP1, JP2, JP3, JP4, JP5, JP6, JP7, JP8: Device_Jumper_NO_Small, KLOR:Jumper, symbol KLORlib:Device_Jumper_NO_Small
- removed OLED1: SSD1306, ScottoKeebs_Components:OLED_128x32, symbol SSD1306-128x64_OLED:SSD1306
- removed PAD+1: +, ScottoKeebs_Scotto:Battery, symbol Mechanical:MountingHole_Pad
- removed PAD-1: -, TOTEMlib:BatteryPad, symbol Mechanical:MountingHole_Pad
- removed SW21: SW_Push, WillKeebs_Kicad_Gateron:SW_MXchoc_HS_1u, symbol Switch:SW_Push
- removed U1: Seeeduino Xiao nRF52840, PCM_marbastlib-xp-promicroish:Xiao_nRF52840_ACH, symbol PCM_marbastlib-promicroish:Seeeduino_Xiao_nRF52840
- added BT1: Pads, willkeebs_power:Battery_Pad, symbol Device:Battery_Cell
- added J2: Conn_01x07_Socket, symbol Connector:Conn_01x07_Socket
- added RES1: RotaryEncoder_Switch, willkeebs_peripherals:RotaryEncoder_Alps_EC11E-Switch_Vertical_H20mm-keebio_modified, symbol Device:RotaryEncoder_Switch
- added U2: ER_OLEDM0.91_1x-I2C, Display:ER_OLEDM0.91_1x-I2C, symbol Display_Graphic:ER_OLEDM0.91_1x-I2C
- added U3: XIAO-nRF52840-Plus-SMD, Seeed_Studio_XIAO_Series:XIAO-nRF52840-Plus-SMD, symbol Seeed_Studio_XIAO_Series:XIAO-nRF52840_Plus_SMD
- JST1: footprint Connector_JST:JST_GH_SM02B-GHS-TB_1x02-1MP_P1.25mm_Horizontal -> willkeebs_power:JST_1.25mm
- PSW1: footprint Button_Switch_SMD:SW_SPDT_Shouhan_MSK12C02 -> willkeebs_power:Switch_MSK12C02
- RSW1: footprint Button_Switch_SMD:SW_Push_1P1T_XKB_TS-1187A -> willkeebs_components:SW_Push_1P1T_XKB_TS-1187A
- SW1, SW10, SW11, SW12, SW13, SW14, SW15, SW16, SW17, SW18, SW19, SW2, SW20, SW3, SW4, SW5, SW6, SW7, SW8, SW9: footprint WillKeebs_Kicad_Gateron:SW_MXchoc_HS_1u -> willkeebs_keyboard:SW_MX_Choc_Hotswap
Connections:
- net +3V3: now also J2.4 (Pin_4), U2.2 (VCC), U3.12 (3V3_OUT)
- net BAT+: now also U3.28 (VBAT)
- net GND: now also BT1.2 (-), J2.5 (Pin_5), RES1.C, U2.1 (GND), U3.13 (GND), U3.27 (GND)
- net LED: now also U3.11 (D10_MOSI)
- net RESET: now also U3.26 (RST)
- net SCL: now also U2.3 (SCL), U3.6 (D5_SCL)
- net SDA: now also U2.4 (SDA), U3.5 (D4_SDA)
- net col0: now also U3.7 (D6_TX)
- net col1: now also U3.15 (D11_SD)
- net col2: now also RES1.S1, U3.16 (D12_SCK)
- net col3: now also U3.17 (D13_WS)
- net col4: now also U3.18 (D14_NFC1)
- net col5: now also U3.8 (D7_RX)
- net row0: now also U3.1 (D0); no longer D25.1 (K)
- net row1: now also U3.2 (D1)
- net row2: now also U3.3 (D2)
- net row3: now also D25.1 (K), U3.4 (D3)
- net at TP1.1: now also U3.24 (SWDIO)
- net at TP2.1: now also U3.25 (SWDCLK)
- net at D25.2 (A): now also RES1.S2
- net at JST1.1 (Pin_1), PSW1.3 (C): now also BT1.1 (+)
- new net BAT-: U3.29 (GND)
- new net D18: J2.7 (Pin_7), U3.22 (D18_MISO)
- new net D8: J2.1 (Pin_1), U3.9 (D8_SCK)
- new net D9: J2.6 (Pin_6), U3.10 (D9_MISO)
- new net ENCA: RES1.A, U3.19 (D15_NFC2)
- new net ENCB: RES1.B, U3.20 (D16)
- new net MOSI: J2.2 (Pin_2), U3.23 (D19_MOSI)
- new net SCK: J2.3 (Pin_3), U3.21 (D17_SCK)
Other:
- note added: "EXTENSION"
- note added: "POWER"
- note removed: "LED should be connected to MOSI pin for the status system"
- note removed: "MCU: Seeed Studio XIAO nRF52840 Firmware: ZMK Matrix: 4×6 Display: SSD1306 (I²C) LED: WS2812B ×3 Power: Single-cell LiPo"
- note removed: "Power Managment"
- moved on the sheet: JST1, MH1, MH2, MH3, MH4, PSW1, TP1, TP2
