File: keyboard/kicad/revisions/dormin-rev_1.0/dormin.kicad_pcb (KiCad board)
At the start: 2 copper layers, 288.7 x 103.4 mm, 44 parts, among them SW1 SW_Push, SW10 SW_Push, SW11 SW_Push, SW12 SW_Push, SW13 SW_Push, SW14 SW_Push, SW15 SW_Push, SW16 SW_Push, SW17 SW_Push, SW18 SW_Push, SW19 SW_Push, SW2 SW_Push, SW20 SW_Push, SW21 SW_Push, SW22 SW_Push, SW23 SW_Push, SW24 SW_Push, SW25 SW_Push, SW26 SW_Push, SW27 SW_Push, SW28 SW_Push, SW29 SW_Push, SW3 SW_Push, SW30 SW_Push, SW31 SW_Push, SW32 SW_Push, SW33 SW_Push, SW34 SW_Push, SW35 SW_Push, SW36 SW_Push, SW37 SW_Push, SW38 SW_Push, SW39 SW_Push, SW4 SW_Push, SW40 SW_Push, SW5 SW_Push, SW6 SW_Push, SW7 SW_Push, SW8 SW_Push, SW9 SW_Push

Commit message: feat: added initial components to the right places
Parts:
- added BT1: Pads, willkeebs_power:Battery_Pad, B.Cu at (190.1, 156.2)
- added BT2_R1: Pads, willkeebs_power:Battery_Pad, F.Cu at (223.4, 156.1)
- added C1: 10uF, Capacitor_SMD:C_0603_1608Metric, B.Cu at (185.8, 119.4)
- added C2: 100nF, Capacitor_SMD:C_0603_1608Metric, B.Cu at (187.5, 119.4)
- added C3: 10uF, Capacitor_SMD:C_0603_1608Metric, F.Cu at (68.1, 106.7)
- added C4: 100nF, Capacitor_SMD:C_0603_1608Metric, F.Cu at (68.1, 108.8)
- added C5_R1: 10uF, Capacitor_SMD:C_0603_1608Metric, B.Cu at (335.4, 96.5)
- added C6_R1: 100nF, Capacitor_SMD:C_0603_1608Metric, B.Cu at (339.1, 96.5)
- added C7_R1: 10uF, Capacitor_SMD:C_0603_1608Metric, B.Cu at (231.9, 119.6)
- added C8_R1: 100nF, Capacitor_SMD:C_0603_1608Metric, B.Cu at (233.9, 119.6)
- added D1: 1N4148W, Diode_SMD:D_SOD-123, F.Cu at (81.9, 128.8)
- added D10: 1N4148W, Diode_SMD:D_SOD-123, F.Cu at (138.9, 109.7)
- added D11: 1N4148W, Diode_SMD:D_SOD-123, F.Cu at (138.9, 90.8)
- added D12: 1N4148W, Diode_SMD:D_SOD-123, F.Cu at (158.0, 133.7)
- added D13: 1N4148W, Diode_SMD:D_SOD-123, F.Cu at (157.9, 114.5)
- added D14: 1N4148W, Diode_SMD:D_SOD-123, F.Cu at (157.9, 95.3)
- added D15: 1N4148W, Diode_SMD:D_SOD-123, F.Cu at (176.9, 138.3)
- added D16: 1N4148W, Diode_SMD:D_SOD-123, F.Cu at (176.8, 119.4)
- added D17: 1N4148W, Diode_SMD:D_SOD-123, F.Cu at (164.0, 104.0)
- added D18: 1N4148W, Diode_SMD:D_SOD-123, F.Cu at (155.8, 158.6)
- added D19: 1N4148W, Diode_SMD:D_SOD-123, F.Cu at (178.6, 162.2)
- added D2: 1N4148W, Diode_SMD:D_SOD-123, F.Cu at (81.9, 109.9)
- added D20: 1N4148W, Diode_SMD:D_SOD-123, F.Cu at (199.8, 171.6)
- added D21: SK6812MINI-E, LED_SMD:LED_SK6812MINI-E_3.2x2.8mm_P1.5mm_ReverseMount, B.Cu at (68.4, 101.1)
- added D22: SK6812MINI-E, LED_SMD:LED_SK6812MINI-E_3.2x2.8mm_P1.5mm_ReverseMount, B.Cu at (73.3, 101.1)
- added D23: SK6812MINI-E, LED_SMD:LED_SK6812MINI-E_3.2x2.8mm_P1.5mm_ReverseMount, B.Cu at (78.2, 101.1)
- added D24: SK6812MINI-E, LED_SMD:LED_SK6812MINI-E_3.2x2.8mm_P1.5mm_ReverseMount, B.Cu at (83.0, 101.1)
- added D25: LED, willkeebs_components:LED_MHT151WDT, F.Cu at (81.6, 159.2)
- added D26: LED, willkeebs_components:LED_MHT151WDT, F.Cu at (81.6, 163.7)
- added D27: D_Schottky, Diode_SMD:D_SOD-523, B.Cu at (196.1, 133.4)
- added D28: KPESD5V0S1UL, Diode_SMD:D_SOD-882, B.Cu at (195.6, 135.1)
- added D29: LED, willkeebs_components:LED_MHT151WDT, F.Cu at (81.6, 168.3)
- added D3: 1N4148W, Diode_SMD:D_SOD-123, F.Cu at (100.4, 138.5)
- added D30: LED, willkeebs_components:LED_MHT151WDT, F.Cu at (81.6, 172.8)
- added D31: LED, willkeebs_components:LED_MHT151WDT, F.Cu at (81.6, 177.3)
- added D32: LED, willkeebs_components:LED_MHT151WDT, F.Cu at (87.3, 159.2)
- added D33: LED, willkeebs_components:LED_MHT151WDT, F.Cu at (87.3, 163.7)
- added D34: LED, willkeebs_components:LED_MHT151WDT, F.Cu at (87.3, 168.3)
- added D35: LED, willkeebs_components:LED_MHT151WDT, F.Cu at (87.3, 172.8)
- added D36: LED, willkeebs_components:LED_MHT151WDT, F.Cu at (87.3, 177.3)
- added D37: LED, willkeebs_components:LED_MHT151WDT, F.Cu at (92.9, 159.2)
- added D38: LED, willkeebs_components:LED_MHT151WDT, F.Cu at (92.9, 163.7)
- added D39: LED, willkeebs_components:LED_MHT151WDT, F.Cu at (92.9, 168.3)
- added D4: 1N4148W, Diode_SMD:D_SOD-123, F.Cu at (100.4, 119.4)
- added D40: LED, willkeebs_components:LED_MHT151WDT, F.Cu at (92.9, 172.8)
- added D41: LED, willkeebs_components:LED_MHT151WDT, F.Cu at (92.9, 177.3)
- added D42: LED, willkeebs_components:LED_MHT151WDT, F.Cu at (98.6, 159.2)
- added D43: LED, willkeebs_components:LED_MHT151WDT, F.Cu at (98.6, 163.7)
- added D44: LED, willkeebs_components:LED_MHT151WDT, F.Cu at (98.6, 168.3)
- added D45: LED, willkeebs_components:LED_MHT151WDT, F.Cu at (98.6, 172.8)
- added D46: LED, willkeebs_components:LED_MHT151WDT, F.Cu at (98.6, 177.3)
- added D47_R1: SK6812MINI-E, LED_SMD:LED_SK6812MINI-E_3.2x2.8mm_P1.5mm_ReverseMount, B.Cu at (335.8, 101.4)
- added D47_R2: D_Schottky, Diode_SMD:D_SOD-523, B.Cu at (220.9, 133.1)
- added D48_R1: SK6812MINI-E, LED_SMD:LED_SK6812MINI-E_3.2x2.8mm_P1.5mm_ReverseMount, B.Cu at (340.7, 101.4)
- added D48_R2: KPESD5V0S1UL, Diode_SMD:D_SOD-882, B.Cu at (220.5, 134.8)
- added D5: 1N4148W, Diode_SMD:D_SOD-123, F.Cu at (100.4, 100.2)
- added D50_R1: SK6812MINI-E, LED_SMD:LED_SK6812MINI-E_3.2x2.8mm_P1.5mm_ReverseMount, B.Cu at (345.6, 101.4)
- added D52_R1: SK6812MINI-E, LED_SMD:LED_SK6812MINI-E_3.2x2.8mm_P1.5mm_ReverseMount, B.Cu at (350.4, 101.4)
- added D53_R1: LED, willkeebs_components:LED_MHT151WDT, F.Cu at (323.3, 161.5)
- added D54_R1: LED, willkeebs_components:LED_MHT151WDT, F.Cu at (323.3, 166.0)
- added D55_R1: LED, willkeebs_components:LED_MHT151WDT, F.Cu at (323.3, 170.6)
- added D56_R1: LED, willkeebs_components:LED_MHT151WDT, F.Cu at (323.3, 175.1)
- added D57_R1: LED, willkeebs_components:LED_MHT151WDT, F.Cu at (323.3, 179.6)
- added D58_R1: LED, willkeebs_components:LED_MHT151WDT, F.Cu at (328.9, 161.5)
- added D59_R1: LED, willkeebs_components:LED_MHT151WDT, F.Cu at (328.9, 166.0)
- added D6: 1N4148W, Diode_SMD:D_SOD-123, F.Cu at (119.6, 133.7)
- added D60_R1: LED, willkeebs_components:LED_MHT151WDT, F.Cu at (328.9, 170.6)
- added D61_R1: 1N4148W, Diode_SMD:D_SOD-123, F.Cu at (294.1, 162.2)
- added D62_R1: 1N4148W, Diode_SMD:D_SOD-123, F.Cu at (294.1, 165.5)
- added D63_R1: 1N4148W, Diode_SMD:D_SOD-123, F.Cu at (294.1, 168.9)
- added D64_R1: 1N4148W, Diode_SMD:D_SOD-123, F.Cu at (294.1, 172.2)
- added D65_R1: LED, willkeebs_components:LED_MHT151WDT, F.Cu at (328.9, 175.1)
- added D66_R1: LED, willkeebs_components:LED_MHT151WDT, F.Cu at (328.9, 179.6)
- added D67_R1: LED, willkeebs_components:LED_MHT151WDT, F.Cu at (334.6, 161.5)
- added D68_R1: LED, willkeebs_components:LED_MHT151WDT, F.Cu at (334.6, 166.0)
- added D69_R1: LED, willkeebs_components:LED_MHT151WDT, F.Cu at (334.6, 170.6)
- added D7: 1N4148W, Diode_SMD:D_SOD-123, F.Cu at (120.1, 114.6)
- added D70_R1: LED, willkeebs_components:LED_MHT151WDT, F.Cu at (334.6, 175.1)
- added D71_R1: LED, willkeebs_components:LED_MHT151WDT, F.Cu at (334.6, 179.6)
- added D72_R1: 1N4148W, Diode_SMD:D_SOD-123, F.Cu at (294.1, 175.6)
- added D73_R1: 1N4148W, Diode_SMD:D_SOD-123, F.Cu at (299.9, 162.2)
- added D74_R1: 1N4148W, Diode_SMD:D_SOD-123, F.Cu at (299.9, 165.5)
- added D75_R1: 1N4148W, Diode_SMD:D_SOD-123, F.Cu at (299.9, 168.9)
- added D76_R1: LED, willkeebs_components:LED_MHT151WDT, F.Cu at (340.3, 161.5)
- added D77_R1: LED, willkeebs_components:LED_MHT151WDT, F.Cu at (340.3, 166.0)
- added D78_R1: LED, willkeebs_components:LED_MHT151WDT, F.Cu at (340.3, 170.6)
- added D79_R1: LED, willkeebs_components:LED_MHT151WDT, F.Cu at (340.3, 175.1)
- added D8: 1N4148W, Diode_SMD:D_SOD-123, F.Cu at (120.1, 95.4)
- added D80_R1: LED, willkeebs_components:LED_MHT151WDT, F.Cu at (340.3, 179.6)
- added D81_R1: 1N4148W, Diode_SMD:D_SOD-123, F.Cu at (299.9, 172.2)
- added D82_R1: 1N4148W, Diode_SMD:D_SOD-123, F.Cu at (299.9, 175.6)
- added D83_R1: 1N4148W, Diode_SMD:D_SOD-123, F.Cu at (305.7, 162.2)
- added D84_R1: 1N4148W, Diode_SMD:D_SOD-123, F.Cu at (305.7, 165.5)
- added D85_R1: 1N4148W, Diode_SMD:D_SOD-123, F.Cu at (305.7, 168.9)
- added D86_R1: 1N4148W, Diode_SMD:D_SOD-123, F.Cu at (305.7, 172.2)
- added D87_R1: 1N4148W, Diode_SMD:D_SOD-123, F.Cu at (305.7, 175.6)
- added D88_R1: 1N4148W, Diode_SMD:D_SOD-123, F.Cu at (311.5, 162.2)
- added D89_R1: 1N4148W, Diode_SMD:D_SOD-123, F.Cu at (311.5, 165.5)
- added D9: 1N4148W, Diode_SMD:D_SOD-123, F.Cu at (139.0, 128.8)
- added D90_R1: 1N4148W, Diode_SMD:D_SOD-123, F.Cu at (311.5, 168.9)
- added D91_R1: 1N4148W, Diode_SMD:D_SOD-123, F.Cu at (311.5, 172.2)
- added D92_R1: 1N4148W, Diode_SMD:D_SOD-123, F.Cu at (311.5, 175.6)
- added F1: Polyfuse, Fuse:Fuse_1206_3216Metric, B.Cu at (197.0, 131.2)
- added F2_R1: Polyfuse, Fuse:Fuse_1206_3216Metric, B.Cu at (221.9, 130.9)
- added J1: Conn_01x06, willkeebs_misc:SMD_Conn_1x06_P2.54mm_Vertical, F.Cu at (187.8, 144.7)
- added J2: Conn_01x04, Connector_PinSocket_2.54mm:PinSocket_1x04_P2.54mm_Vertical, F.Cu at (190.3, 141.0)
- added J3: Conn_01x02, willkeebs_misc:SMD_Conn_1x02_P2.54mm_Vertical, F.Cu at (204.1, 131.4)
- added J4_R1: Conn_01x06, willkeebs_misc:SMD_Conn_1x06_P2.54mm_Vertical, F.Cu at (219.1, 144.7)
- added J4_R2: Conn_01x02, willkeebs_misc:SMD_Conn_1x02_P2.54mm_Vertical, B.Cu at (214.9, 131.4)
- added J6_R1: Conn_01x04, Connector_PinSocket_2.54mm:PinSocket_1x04_P2.54mm_Vertical, F.Cu at (221.7, 141.1)
- added JST1: Conn_01x02_Pin, Connector_JST:JST_GH_SM02B-GHS-TB_1x02-1MP_P1.25mm_Horizontal, B.Cu at (197.3, 156.1)
- added JST2_R1: Conn_01x02_Pin, Connector_JST:JST_GH_SM02B-GHS-TB_1x02-1MP_P1.25mm_Horizontal, B.Cu at (218.1, 156.1)
- added MH1: MountingHole_2.2mm_M2, MountingHole:MountingHole_2.2mm_M2, F.Cu at (85.8, 113.4)
- added MH2: MountingHole_2.2mm_M2, MountingHole:MountingHole_2.2mm_M2, F.Cu at (86.1, 143.0)
- added MH3: MountingHole_2.2mm_M2, MountingHole:MountingHole_2.2mm_M2, F.Cu at (163.2, 115.2)
- added MH4: MountingHole_2.2mm_M2, MountingHole:MountingHole_2.2mm_M2, F.Cu at (162.4, 155.3)
- added MH5_R1: MountingHole_2.2mm_M2, MountingHole:MountingHole_2.2mm_M2, F.Cu at (332.6, 115.6)
- added MH6_R1: MountingHole_2.2mm_M2, MountingHole:MountingHole_2.2mm_M2, F.Cu at (333.3, 135.3)
- added MH7_R1: MountingHole_2.2mm_M2, MountingHole:MountingHole_2.2mm_M2, F.Cu at (257.5, 113.2)
- added MH8_R1: MountingHole_2.2mm_M2, MountingHole:MountingHole_2.2mm_M2, F.Cu at (256.8, 155.0)
- added PSW1: SW_SPDT, PCM_marbastlib-various:SW_MSK12C02-HB, B.Cu at (178.3, 96.1)
- added PSW2_R1: SW_SPDT, PCM_marbastlib-various:SW_MSK12C02-HB, B.Cu at (240.9, 96.1)
- added Q1: AO3400A, Package_TO_SOT_SMD:SOT-23, B.Cu at (201.8, 123.6)
- added Q2: AO3407A, Package_TO_SOT_SMD:SOT-23, B.Cu at (193.2, 123.6)
- added Q3_R1: AO3407A, Package_TO_SOT_SMD:SOT-23, B.Cu at (219.7, 123.6)
- added Q4_R1: AO3400A, Package_TO_SOT_SMD:SOT-23, B.Cu at (227.5, 123.5)
- added R1: 1K, Resistor_SMD:R_0603_1608Metric, F.Cu at (109.0, 169.0)
- added R10: 1K, Resistor_SMD:R_0603_1608Metric, F.Cu at (113.0, 166.5)
- added R11: 1K, Resistor_SMD:R_0603_1608Metric, F.Cu at (113.0, 169.0)
- added R12: 1K, Resistor_SMD:R_0603_1608Metric, F.Cu at (113.0, 171.5)
- added R13: 1K, Resistor_SMD:R_0603_1608Metric, F.Cu at (113.0, 174.0)
- added R14: 1K, Resistor_SMD:R_0603_1608Metric, F.Cu at (113.0, 176.5)
- added R15: 1K, Resistor_SMD:R_0603_1608Metric, F.Cu at (117.0, 159.0)
- added R16: 1K, Resistor_SMD:R_0603_1608Metric, F.Cu at (117.0, 161.5)
- added R17: 1K, Resistor_SMD:R_0603_1608Metric, F.Cu at (117.0, 164.0)
- added R18: 1K, Resistor_SMD:R_0603_1608Metric, F.Cu at (117.0, 166.5)
- added R19: 1K, Resistor_SMD:R_0603_1608Metric, F.Cu at (117.0, 169.0)
- added R2: 1K, Resistor_SMD:R_0603_1608Metric, F.Cu at (109.0, 171.5)
- added R20: 1K, Resistor_SMD:R_0603_1608Metric, F.Cu at (117.0, 171.5)
- added R21: 1K, Resistor_SMD:R_0603_1608Metric, F.Cu at (117.0, 174.0)
- added R22: 1K, Resistor_SMD:R_0603_1608Metric, F.Cu at (117.0, 176.5)
- added R25_R1: 1K, Resistor_SMD:R_0603_1608Metric, F.Cu at (351.3, 170.3)
- added R26_R1: 1K, Resistor_SMD:R_0603_1608Metric, F.Cu at (351.3, 172.8)
- added R27_R1: 1K, Resistor_SMD:R_0603_1608Metric, F.Cu at (351.3, 175.3)
- added R28_R1: 1K, Resistor_SMD:R_0603_1608Metric, F.Cu at (351.3, 177.8)
- added R29_R1: 1K, Resistor_SMD:R_0603_1608Metric, F.Cu at (355.3, 160.3)
- added R3: 1K, Resistor_SMD:R_0603_1608Metric, F.Cu at (109.0, 174.0)
- added R30_R1: 1K, Resistor_SMD:R_0603_1608Metric, F.Cu at (355.3, 162.8)
- added R31_R1: 1K, Resistor_SMD:R_0603_1608Metric, F.Cu at (355.3, 165.3)
- added R32_R1: 1K, Resistor_SMD:R_0603_1608Metric, F.Cu at (355.3, 167.8)
- added R33_R1: 1K, Resistor_SMD:R_0603_1608Metric, F.Cu at (355.3, 170.3)
- added R34_R1: 1K, Resistor_SMD:R_0603_1608Metric, F.Cu at (355.3, 172.8)
- added R35_R1: 1K, Resistor_SMD:R_0603_1608Metric, F.Cu at (355.3, 175.3)
- added R36_R1: 1K, Resistor_SMD:R_0603_1608Metric, F.Cu at (355.3, 177.8)
- added R37_R1: 1K, Resistor_SMD:R_0603_1608Metric, F.Cu at (359.3, 160.3)
- added R38_R1: 1K, Resistor_SMD:R_0603_1608Metric, F.Cu at (359.3, 162.8)
- added R39_R1: 1K, Resistor_SMD:R_0603_1608Metric, F.Cu at (359.3, 165.3)
- added R4: 1K, Resistor_SMD:R_0603_1608Metric, F.Cu at (109.0, 176.5)
- added R40_R1: 1K, Resistor_SMD:R_0603_1608Metric, F.Cu at (359.3, 167.8)
- added R41_R1: 1K, Resistor_SMD:R_0603_1608Metric, F.Cu at (359.3, 170.3)
- added R42_R1: 1K, Resistor_SMD:R_0603_1608Metric, F.Cu at (359.3, 172.8)
- added R43_R1: 1K, Resistor_SMD:R_0603_1608Metric, F.Cu at (359.3, 175.3)
- added R44_R1: 1K, Resistor_SMD:R_0603_1608Metric, F.Cu at (359.3, 177.8)
- added R7: 1K, Resistor_SMD:R_0603_1608Metric, F.Cu at (113.0, 159.0)
- added R706: 100R, Resistor_SMD:R_0603_1608Metric, B.Cu at (202.7, 119.5)
- added R707: 10k, Resistor_SMD:R_0603_1608Metric, B.Cu at (200.9, 119.5)
- added R708_R1: 100R, Resistor_SMD:R_0603_1608Metric, B.Cu at (226.4, 119.5)
- added R709_R1: 10k, Resistor_SMD:R_0603_1608Metric, B.Cu at (228.6, 119.5)
- added R710: 100R, Resistor_SMD:R_0603_1608Metric, B.Cu at (191.7, 119.5)
- added R711: 100k, Resistor_SMD:R_0603_1608Metric, B.Cu at (194.6, 119.5)
- added R712: 330R, Resistor_SMD:R_0603_1608Metric, B.Cu at (205.6, 105.0)
- added R713_R1: 100R, Resistor_SMD:R_0603_1608Metric, F.Cu at (238.1, 107.2)
- added R714_R1: 100k, Resistor_SMD:R_0603_1608Metric, B.Cu at (221.1, 119.2)
- added R715_R1: 330R, Resistor_SMD:R_0603_1608Metric, B.Cu at (218.6, 119.2)
- added R8: 1K, Resistor_SMD:R_0603_1608Metric, F.Cu at (113.0, 161.5)
- added R9: 1K, Resistor_SMD:R_0603_1608Metric, F.Cu at (113.0, 164.0)
- added RSW1: RSW1, Button_Switch_SMD:SW_SPST_SKQG_WithStem, B.Cu at (139.6, 157.7)
- added RSW2_R1: RSW1, Button_Switch_SMD:SW_SPST_SKQG_WithStem, B.Cu at (279.0, 157.7)
- added TP1: VBAT, TestPoint:TestPoint_Pad_D1.0mm, F.Cu at (71.6, 148.5)
- added TP2: GND, TestPoint:TestPoint_Pad_D1.0mm, F.Cu at (74.6, 148.5)
- added TP3: STS_LED_EN, TestPoint:TestPoint_Pad_D1.0mm, F.Cu at (77.7, 148.5)
- added TP4_R1: VBAT_R, TestPoint:TestPoint_Pad_D1.0mm, F.Cu at (341.9, 149.4)
- added TP5_R1: GND, TestPoint:TestPoint_Pad_D1.0mm, F.Cu at (345.0, 149.4)
- added TP6_R1: STS_LED_EN_R, TestPoint:TestPoint_Pad_D1.0mm, F.Cu at (348.1, 149.4)
- added U3: XIAO-nRF52840-Plus-SMD, Seeed_Studio_XIAO_Series:XIAO-nRF52840-Plus-SMD, B.Cu at (193.9, 105.1)
- added U5_R1: XIAO-nRF52840-Plus-SMD, Seeed_Studio_XIAO_Series:XIAO-nRF52840-Plus-SMD, B.Cu at (225.2, 105.1)
- SW1, SW10, SW11, SW12, SW13, SW14, SW15, SW16, SW17, SW18, SW19, SW2, SW20, SW21, SW22, SW23, SW24, SW25, SW26, SW27, SW28, SW29, SW3, SW30, SW31, SW32, SW33, SW34, SW35, SW36, SW37, SW38, SW39, SW4, SW40, SW5, SW6, SW7, SW8, SW9: footprint SW_MX_Choc_Hotswap -> willkeebs_keyboard:NF_LED_1206_SW_KS33_3_0_HS_1U
- turned SW1 to 180 degrees
- turned SW10 to 180 degrees
- turned SW11 to 180 degrees
- turned SW12 to 180 degrees
- turned SW13 to 180 degrees
- turned SW14 to 180 degrees
- turned SW15 to 180 degrees
- turned SW16 to 180 degrees
- turned SW17 to 180 degrees
- turned SW18 to 180 degrees
- turned SW19 to 165 degrees
- turned SW2 to 180 degrees
- turned SW20 to 151 degrees
- turned SW21 to 180 degrees
- turned SW22 to 180 degrees
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Connections:
- SW1 pad 1: outer_home_from -> Net-(D1-A)
- SW1 pad 2: outer_home_to -> COL5
- SW10 pad 1: middle_home_from -> Net-(D10-A)
- SW10 pad 2: middle_home_to -> COL1
- SW11 pad 1: middle_top_from -> Net-(D11-A)
- SW11 pad 2: middle_top_to -> COL0
- SW12 pad 1: index_bottom_from -> Net-(D12-A)
- SW12 pad 2: index_bottom_to -> COL5
- SW13 pad 1: index_home_from -> Net-(D13-A)
- SW13 pad 2: index_home_to -> COL4
- SW14 pad 1: index_top_from -> Net-(D14-A)
- SW14 pad 2: index_top_to -> COL3
- SW15 pad 1: inner_bottom_from -> Net-(D15-A)
- SW15 pad 2: inner_bottom_to -> COL2
- SW16 pad 1: inner_home_from -> Net-(D16-A)
- SW16 pad 2: inner_home_to -> COL1
- SW17 pad 1: inner_top_from -> Net-(D17-A)
- SW17 pad 2: inner_top_to -> COL0
- SW18 pad 1: inner_only_from -> Net-(D18-A)
- SW18 pad 2: inner_only_to -> COL5
- SW19 pad 1: home_only_from -> Net-(D19-A)
- SW19 pad 2: home_only_to -> COL4
- SW2 pad 1: outer_top_from -> Net-(D2-A)
- SW2 pad 2: outer_top_to -> COL4
- SW20 pad 1: outer_only_from -> Net-(D20-A)
- SW20 pad 2: outer_only_to -> COL3
- SW21 pad 1: mirror_outer_home_from -> Net-(D61_R1-A)
- SW21 pad 2: mirror_outer_home_to -> COL5_R
- SW22 pad 1: mirror_outer_top_from -> Net-(D62_R1-A)
- SW22 pad 2: mirror_outer_top_to -> COL5_R
- SW23 pad 1: mirror_pinky_bottom_from -> Net-(D63_R1-A)
- SW23 pad 2: mirror_pinky_bottom_to -> COL5_R
- SW24 pad 1: mirror_pinky_home_from -> Net-(D64_R1-A)
- SW24 pad 2: mirror_pinky_home_to -> COL5_R
- SW25 pad 1: mirror_pinky_top_from -> Net-(D72_R1-A)
- SW25 pad 2: mirror_pinky_top_to -> COL4_R
- SW26 pad 1: mirror_ring_bottom_from -> Net-(D73_R1-A)
- SW26 pad 2: mirror_ring_bottom_to -> COL4_R
- SW27 pad 1: mirror_ring_home_from -> Net-(D74_R1-A)
- SW27 pad 2: mirror_ring_home_to -> COL4_R
- SW28 pad 1: mirror_ring_top_from -> Net-(D75_R1-A)
- SW28 pad 2: mirror_ring_top_to -> COL4_R
- SW29 pad 1: mirror_middle_bottom_from -> Net-(D81_R1-A)
- SW29 pad 2: mirror_middle_bottom_to -> COL3_R
- SW3 pad 1: pinky_bottom_from -> Net-(D3-A)
- SW3 pad 2: pinky_bottom_to -> COL3
- SW30 pad 1: mirror_middle_home_from -> Net-(D82_R1-A)
- SW30 pad 2: mirror_middle_home_to -> COL3_R
- SW31 pad 1: mirror_middle_top_from -> Net-(D83_R1-A)
- SW31 pad 2: mirror_middle_top_to -> COL3_R
- SW32 pad 1: mirror_index_bottom_from -> Net-(D84_R1-A)
- SW32 pad 2: mirror_index_bottom_to -> COL3_R
- SW33 pad 1: mirror_index_home_from -> Net-(D85_R1-A)
- SW33 pad 2: mirror_index_home_to -> COL2_R
- SW34 pad 1: mirror_index_top_from -> Net-(D86_R1-A)
- SW34 pad 2: mirror_index_top_to -> COL2_R
- SW35 pad 1: mirror_inner_bottom_from -> Net-(D87_R1-A)
- SW35 pad 2: mirror_inner_bottom_to -> COL2_R
- SW36 pad 1: mirror_inner_home_from -> Net-(D88_R1-A)
- SW36 pad 2: mirror_inner_home_to -> COL1_R
- SW37 pad 1: mirror_inner_top_from -> Net-(D89_R1-A)
- SW37 pad 2: mirror_inner_top_to -> COL1_R
- SW38 pad 1: mirror_inner_only_from -> Net-(D90_R1-A)
- SW38 pad 2: mirror_inner_only_to -> COL1_R
- SW39 pad 1: mirror_home_only_from -> Net-(D91_R1-A)
- SW39 pad 2: mirror_home_only_to -> COL0_R
- SW4 pad 1: pinky_home_from -> Net-(D4-A)
- SW4 pad 2: pinky_home_to -> COL2
- SW40 pad 1: mirror_outer_only_from -> Net-(D92_R1-A)
- SW40 pad 2: mirror_outer_only_to -> COL0_R
- SW5 pad 1: pinky_top_from -> Net-(D5-A)
- SW5 pad 2: pinky_top_to -> COL1
- SW6 pad 1: ring_bottom_from -> Net-(D6-A)
- SW6 pad 2: ring_bottom_to -> COL5
- SW7 pad 1: ring_home_from -> Net-(D7-A)
- SW7 pad 2: ring_home_to -> COL4
- SW8 pad 1: ring_top_from -> Net-(D8-A)
- SW8 pad 2: ring_top_to -> COL3
- SW9 pad 1: middle_bottom_from -> Net-(D9-A)
- SW9 pad 2: middle_bottom_to -> COL2

Commit message: feat: placed components for the left half
Parts:
- BT2_R1, C3, C4, D1, D10, D11, D12, D13, D14, D15, D16, D17, D18, D19, D2, D20, D25, D26, D29, D3, D30, D31, D32, D33, D34, D35, D36, D37, D38, D39, D4, D40, D41, D42, D43, D44, D45, D46, D5, D6, D7, D8, D9, R1, R10, R11, R12, R13, R14, R15, R16, R17, R18, R19, R2, R20, R21, R22, R3, R4, R7, R8, R9: moved to B.Cu
- moved R44_R1 140.5 mm to (218.9, 171.7)
- moved R41_R1 135.9 mm to (242.8, 100.3)
- moved R40_R1 126.0 mm to (242.9, 119.5)
- moved R43_R1 119.7 mm to (240.3, 162.4)
- moved R39_R1 119.6 mm to (242.8, 138.6)
- moved R38_R1 118.4 mm to (261.9, 95.4)
- moved D80_R1 117.5 mm to (223.3, 169.3)
- moved D77_R1 113.9 mm to (247.3, 100.2)
- moved R35_R1 112.4 mm to (281.1, 90.8)
- moved R37_R1 107.5 mm to (262.0, 114.6)
- moved D70_R1 105.0 mm to (266.2, 95.4)
- moved R36_R1 103.0 mm to (262.2, 133.8)
- moved D76_R1 102.3 mm to (247.1, 119.4)
- moved R34_R1 97.5 mm to (280.9, 109.8)
- moved D40 97.3 mm to (152.1, 95.5)
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
Commit message: feat: finish pcbs component placements
Parts:
- D53_R1, D54_R1, D55_R1, D56_R1, D57_R1, D58_R1, D59_R1, D60_R1, D61_R1, D62_R1, D63_R1, D64_R1, D65_R1, D66_R1, D67_R1, D68_R1, D69_R1, D70_R1, D71_R1, D72_R1, D73_R1, D74_R1, D75_R1, D76_R1, D77_R1, D78_R1, D79_R1, D80_R1, D81_R1, D82_R1, D83_R1, D84_R1, D85_R1, D86_R1, D87_R1, D88_R1, D89_R1, D90_R1, D91_R1, D92_R1, R25_R1, R26_R1, R27_R1, R28_R1, R29_R1, R30_R1, R31_R1, R32_R1, R33_R1, R34_R1, R35_R1, R36_R1, R37_R1, R38_R1, R39_R1, R40_R1, R41_R1, R42_R1, R43_R1, R44_R1, R713_R1: moved to B.Cu
- moved R41_R1 13.0 mm to (255.3, 103.8), turned to -90 degrees
- moved MH2 9.00 mm to (85.8, 134.0)
- moved R713_R1 3.32 mm to (236.1, 109.9), turned to -90 degrees
- moved MH7_R1 1.81 mm to (257.1, 115.0)
- moved RSW1 1.64 mm to (139.6, 156.1)
- moved MH1 1.36 mm to (85.8, 114.7)
- moved R44_R1 1.27 mm to (220.1, 172.2), turned to -151 degrees
- moved MH3 1.26 mm to (162.0, 115.0)
- moved MH6_R1 1.20 mm to (333.4, 134.1)
- moved MH5_R1 1.03 mm to (333.4, 114.9)
- moved D80_R1 0.98 mm to (224.1, 169.9), turned to 29 degrees
- moved D14 0.82 mm to (157.3, 95.6)
- moved D58_R1 0.74 mm to (304.5, 133.6)
- moved R43_R1 0.71 mm to (241.0, 162.6), turned to -165 degrees
- moved D13 0.71 mm to (157.3, 114.7)
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Other:
- board text added: "3V3"
- board text added: "EXTA"
- board text added: "EXTB"
- board text added: "GND"
- board text added: "SCL"
- board text added: "SDA"
- board text added: "SWC"
- board text added: "SWD"

Commit message: feat: adjust schematics for the switches logic order
Connections:
- D1 pad 1: ROW0 -> ROW2
- D11 pad 1: ROW1 -> ROW0
- D13 pad 1: ROW2 -> ROW1
- D14 pad 1: ROW2 -> ROW0
- D16 pad 1: ROW2 -> ROW1
- D17 pad 1: ROW2 -> ROW0
- D2 pad 1: ROW0 -> ROW1
- D3 pad 1: ROW0 -> ROW2
- D4 pad 1: ROW0 -> ROW1
- D6 pad 1: ROW1 -> ROW2
- D61_R1 pad 1: ROW0_R -> ROW2_R
- D64_R1 pad 1: ROW3_R -> ROW1_R
- D73_R1 pad 1: ROW1_R -> ROW2_R
- D74_R1 pad 1: ROW2_R -> ROW1_R
- D75_R1 pad 1: ROW3_R -> ROW0_R
- D8 pad 1: ROW1 -> ROW0
- D81_R1 pad 1: ROW0_R -> ROW2_R
- D83_R1 pad 1: ROW2_R -> ROW0_R
- D84_R1 pad 1: ROW3_R -> ROW2_R
- D85_R1 pad 1: ROW0_R -> ROW1_R
- D86_R1 pad 1: ROW1_R -> ROW0_R
- D88_R1 pad 1: ROW0_R -> ROW1_R
- D89_R1 pad 1: ROW1_R -> ROW0_R
- D9 pad 1: ROW1 -> ROW2
- D90_R1 pad 1: ROW2_R -> ROW3_R
- D91_R1 pad 1: ROW1_R -> ROW3_R
- D92_R1 pad 1: ROW2_R -> ROW3_R
- SW1 pad 2: COL5 -> COL0
- SW10 pad 2: COL1 -> COL3
- SW11 pad 2: COL0 -> COL3
- SW12 pad 2: COL5 -> COL4
- SW14 pad 2: COL3 -> COL4
- SW15 pad 2: COL2 -> COL5
- SW16 pad 2: COL1 -> COL5
- SW17 pad 2: COL0 -> COL5
- SW18 pad 2: COL5 -> COL3
- SW2 pad 2: COL4 -> COL0
- SW20 pad 2: COL3 -> COL5
- SW23 pad 2: COL5_R -> COL4_R
- SW24 pad 2: COL5_R -> COL4_R
- SW26 pad 2: COL4_R -> COL3_R
- SW27 pad 2: COL4_R -> COL3_R
- SW28 pad 2: COL4_R -> COL3_R
- SW29 pad 2: COL3_R -> COL2_R
- SW3 pad 2: COL3 -> COL1
- SW30 pad 2: COL3_R -> COL2_R
- SW31 pad 2: COL3_R -> COL2_R
- SW32 pad 2: COL3_R -> COL1_R
- SW33 pad 2: COL2_R -> COL1_R
- SW34 pad 2: COL2_R -> COL1_R
- SW35 pad 2: COL2_R -> COL0_R
- SW36 pad 2: COL1_R -> COL0_R
- SW37 pad 2: COL1_R -> COL0_R
- SW38 pad 2: COL1_R -> COL0_R
- SW39 pad 2: COL0_R -> COL1_R
- SW4 pad 2: COL2 -> COL1
- SW40 pad 2: COL0_R -> COL2_R
- SW6 pad 2: COL5 -> COL2
- SW7 pad 2: COL4 -> COL2
- SW8 pad 2: COL3 -> COL2
- SW9 pad 2: COL2 -> COL3
Changed lines of the file:
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@@
 			(layers "B.Cu" "B.Mask" "B.Paste")
 			(roundrect_rratio 0.1)
-			(net "COL5")
+			(net "COL4")
 			(pinfunction "2_2")
 			(pintype "passive")
@@
 			(layers "B.Cu" "B.Mask" "B.Paste")
 			(roundrect_rratio 0.1)
-			(net "COL3")
+			(net "COL1")
 			(pinfunction "2_2")
 			(pintype "passive")
@@
 			(layers "B.Cu" "B.Mask" "B.Paste")
 			(roundrect_rratio 0.1)
-			(net "COL4_R")
+			(net "COL3_R")
 			(pinfunction "2_2")
 			(pintype "passive")
@@
 			(layers "B.Cu" "B.Mask" "B.Paste")
 			(roundrect_rratio 0.1)
-			(net "COL1")
+			(net "COL5")
 			(pinfunction "2_2")
 			(pintype "passive")
@@
 			(layers "B.Cu" "B.Mask" "B.Paste")
 			(roundrect_rratio 0.1)
-			(net "COL2_R")
+			(net "COL1_R")
 			(pinfunction "2_2")
 			(pintype "passive")
@@
 			(layers "B.Cu" "B.Mask" "B.Paste")
 			(roundrect_rratio 0.1)
-			(net "COL2")
+			(net "COL1")
 			(pinfunction "2_2")
 			(pintype "passive")
@@
 			(layers "B.Cu" "B.Mask" "B.Paste")
 			(roundrect_rratio 0.1)
-			(net "COL5_R")
+			(net "COL4_R")
 			(pinfunction "2_2")
 			(pintype "passive")
@@
 			(layers "B.Cu" "B.Mask" "B.Paste")
 			(roundrect_rratio 0.1)
-			(net "COL3")
+			(net "COL2")
 			(pinfunction "2_2")
 			(pintype "passive")
@@
 			(layers "B.Cu" "B.Mask" "B.Paste")
 			(roundrect_rratio 0.1)
-			(net "COL3_R")
+			(net "COL2_R")
 			(pinfunction "2_2")
 			(pintype "passive")
@@
 			(layers "B.Cu" "B.Mask" "B.Paste")
 			(roundrect_rratio 0.1)
-			(net "COL0_R")
+			(net "COL2_R")
 			(pinfunction "2_2")
 			(pintype "passive")
@@
 			(layers "B.Cu" "B.Mask" "B.Paste")
 			(roundrect_rratio 0.1)
-			(net "COL2_R")
+			(net "COL1_R")
 			(pinfunction "2_2")
 			(pintype "passive")
@@
 			(layers "B.Cu" "B.Mask" "B.Paste")
 			(roundrect_rratio 0.1)
-			(net "COL3_R")
+			(net "COL2_R")
 			(pinfunction "2_2")
 			(pintype "passive")
@@
 			(layers "B.Cu" "B.Mask" "B.Paste")
 			(roundrect_rratio 0.1)
-			(net "COL3_R")
+			(net "COL1_R")
 			(pinfunction "2_2")
 			(pintype "passive")
@@
 			(layers "B.Cu" "B.Mask" "B.Paste")
 			(roundrect_rratio 0.1)
-			(net "COL5")
+			(net "COL3")
 			(pinfunction "2_2")
 			(pintype "passive")
@@
 			(layers "B.Cu" "B.Mask" "B.Paste")
 			(roundrect_rratio 0.1)
-			(net "COL4_R")
+			(net "COL3_R")
 			(pinfunction "2_2")
 			(pintype "passive")
@@
 			(layers "B.Cu" "B.Mask" "B.Paste")
 			(roundrect_rratio 0.1)
-			(net "COL3")
+			(net "COL4")
 			(pinfunction "2_2")
 			(pintype "passive")
@@
 			(layers "B.Cu" "B.Mask" "B.Paste")
 			(roundrect_rratio 0.1)
-			(net "COL0_R")
+			(net "COL1_R")
 			(pinfunction "2_2")
 			(pintype "passive")
@@
 			(layers "B.Cu" "B.Mask" "B.Paste")
 			(roundrect_rratio 0.1)
-			(net "COL1_R")
+			(net "COL0_R")
 			(pinfunction "2_2")
 			(pintype "passive")
@@
 			(layers "B.Cu" "B.Mask" "B.Paste")
 			(roundrect_rratio 0.1)
-			(net "COL1_R")
+			(net "COL0_R")
 			(pinfunction "2_2")
 			(pintype "passive")
@@
 			(layers "B.Cu" "B.Mask" "B.Paste")
 			(roundrect_rratio 0.1)
-			(net "COL1")
+			(net "COL3")
 			(pinfunction "2_2")
 			(pintype "passive")
@@
 			(layers "B.Cu" "B.Mask" "B.Paste")
 			(roundrect_rratio 0.1)
-			(net "COL3")
+			(net "COL5")
 			(pinfunction "2_2")
 			(pintype "passive")
@@
 			(layers "B.Cu" "B.Mask" "B.Paste")
 			(roundrect_rratio 0.1)
-			(net "COL4")
+			(net "COL2")
 			(pinfunction "2_2")
 			(pintype "passive")
@@
 			(layers "B.Cu" "B.Mask" "B.Paste")
 			(roundrect_rratio 0.1)
-			(net "COL2")
+			(net "COL3")
 			(pinfunction "2_2")
 			(pintype "passive")
@@
 			(layers "B.Cu" "B.Mask" "B.Paste")
 			(roundrect_rratio 0.1)
-			(net "COL1_R")
+			(net "COL0_R")
 			(pinfunction "2_2")
 			(pintype "passive")
@@
 			(layers "B.Cu" "B.Mask" "B.Paste")
 			(roundrect_rratio 0.1)
-			(net "COL4")
+			(net "COL0")
 			(pinfunction "2_2")
 			(pintype "passive")
@@
 			(layers "B.Cu" "B.Mask" "B.Paste")
 			(roundrect_rratio 0.1)
-			(net "COL5")
+			(net "COL0")
 			(pinfunction "2_2")
 			(pintype "passive")
@@
 			(layers "B.Cu" "B.Mask" "B.Paste")
 			(roundrect_rratio 0.1)
-			(net "COL0")
+			(net "COL3")
 			(pinfunction "2_2")
 			(pintype "passive")
@@
 			(layers "B.Cu" "B.Mask" "B.Paste")
 			(roundrect_rratio 0.1)
-			(net "COL0")
+			(net "COL5")
 			(pinfunction "2_2")
 			(pintype "passive")
@@
 			(layers "B.Cu" "B.Mask" "B.Paste")
 			(roundrect_rratio 0.1)
-			(net "COL2_R")
+			(net "COL0_R")
 			(pinfunction "2_2")
 			(pintype "passive")
@@
 			(layers "B.Cu" "B.Mask" "B.Paste")
 			(roundrect_rratio 0.1)
-			(net "COL2")
+			(net "COL5")
 			(pinfunction "2_2")
 			(pintype "passive")
@@
 			(layers "B.Cu" "B.Mask" "B.Paste")
 			(roundrect_rratio 0.1)
-			(net "COL4_R")
+			(net "COL3_R")
 			(pinfunction "2_2")
 			(pintype "passive")
@@
 			(layers "B.Cu" "B.Mask" "B.Paste")
 			(roundrect_rratio 0.1)
-			(net "COL3_R")
+			(net "COL2_R")
 			(pinfunction "2_2")
 			(pintype "passive")
@@
 			(layers "B.Cu" "B.Mask" "B.Paste")
 			(roundrect_rratio 0.1)
-			(net "COL5")
+			(net "COL2")
 			(pinfunction "2_2")
 			(pintype "passive")
@@
 			(layers "B.Cu" "B.Mask" "B.Paste")
 			(roundrect_rratio 0.1)
-			(net "COL5_R")
+			(net "COL4_R")
 			(pinfunction "2_2")
 			(pintype "passive")
@@
 			(layers "B.Cu" "B.Mask" "B.Paste")
 			(roundrect_rratio 0.25)
-			(net "ROW1_R")
+			(net "ROW3_R")
 			(pinfunction "K_1")
 			(pintype "passive")
@@
 			(layers "B.Cu" "B.Mask" "B.Paste")
 			(roundrect_rratio 0.25)
-			(net "ROW0_R")
+			(net "ROW2_R")
 			(pinfunction "K_1")
 			(pintype "passive")
@@
 			(layers "B.Cu" "B.Mask" "B.Paste")
 			(roundrect_rratio 0.25)
-			(net "ROW2_R")
+			(net "ROW0_R")
 			(pinfunction "K_1")
 			(pintype "passive")
@@
 			(layers "B.Cu" "B.Mask" "B.Paste")
 			(roundrect_rratio 0.25)
-			(net "ROW2")
+			(net "ROW1")
 			(pinfunction "K_1")
 			(pintype "passive")
@@
 			(layers "B.Cu" "B.Mask" "B.Paste")
 			(roundrect_rratio 0.25)
-			(net "ROW0")
+			(net "ROW1")
 			(pinfunction "K_1")
 			(pintype "passive")
@@
 			(layers "B.Cu" "B.Mask" "B.Paste")
 			(roundrect_rratio 0.25)
-			(net "ROW3_R")
+			(net "ROW1_R")
 			(pinfunction "K_1")
 			(pintype "passive")
@@
 			(layers "B.Cu" "B.Mask" "B.Paste")
 			(roundrect_rratio 0.25)
-			(net "ROW2_R")
+			(net "ROW3_R")
 			(pinfunction "K_1")
 			(pintype "passive")
@@
 			(layers "B.Cu" "B.Mask" "B.Paste")
 			(roundrect_rratio 0.25)
-			(net "ROW1_R")
+			(net "ROW0_R")
 			(pinfunction "K_1")
 			(pintype "passive")
@@
 			(layers "B.Cu" "B.Mask" "B.Paste")
 			(roundrect_rratio 0.25)
-			(net "ROW2")
+			(net "ROW1")
 			(pinfunction "K_1")
 			(pintype "passive")
@@
 			(layers "B.Cu" "B.Mask" "B.Paste")
 			(roundrect_rratio 0.25)
-			(net "ROW2")
+			(net "ROW0")
 			(pinfunction "K_1")
 			(pintype "passive")
@@
 			(layers "B.Cu" "B.Mask" "B.Paste")
 			(roundrect_rratio 0.25)
-			(net "ROW3_R")
+			(net "ROW0_R")
 			(pinfunction "K_1")
 			(pintype "passive")
@@
 			(layers "B.Cu" "B.Mask" "B.Paste")
 			(roundrect_rratio 0.25)
-			(net "ROW1")
+			(net "ROW2")
 			(pinfunction "K_1")
 			(pintype "passive")
@@
 			(layers "B.Cu" "B.Mask" "B.Paste")
 			(roundrect_rratio 0.25)
-			(net "ROW1")
+			(net "ROW0")
 			(pinfunction "K_1")
 			(pintype "passive")
@@
 			(layers "B.Cu" "B.Mask" "B.Paste")
 			(roundrect_rratio 0.25)
-			(net "ROW0")
+			(net "ROW2")
 			(pinfunction "K_1")
 			(pintype "passive")
@@
 			(layers "B.Cu" "B.Mask" "B.Paste")
 			(roundrect_rratio 0.25)
-			(net "ROW1_R")
+			(net "ROW0_R")
 			(pinfunction "K_1")
 			(pintype "passive")
@@
 			(layers "B.Cu" "B.Mask" "B.Paste")
 			(roundrect_rratio 0.25)
-			(net "ROW2_R")
+			(net "ROW1_R")
 			(pinfunction "K_1")
 			(pintype "passive")
@@
 			(layers "B.Cu" "B.Mask" "B.Paste")
 			(roundrect_rratio 0.25)
-			(net "ROW2")
+			(net "ROW0")
 			(pinfunction "K_1")
 			(pintype "passive")
@@
 			(layers "B.Cu" "B.Mask" "B.Paste")
 			(roundrect_rratio 0.25)
-			(net "ROW0_R")
+			(net "ROW2_R")
 			(pinfunction "K_1")
 			(pintype "passive")
@@
 			(layers "B.Cu" "B.Mask" "B.Paste")
 			(roundrect_rratio 0.25)
-			(net "ROW2_R")
+			(net "ROW3_R")
 			(pinfunction "K_1")
 			(pintype "passive")
@@
 			(layers "B.Cu" "B.Mask" "B.Paste")
 			(roundrect_rratio 0.25)
-			(net "ROW0_R")
+			(net "ROW1_R")
 			(pinfunction "K_1")
 			(pintype "passive")
@@
 			(layers "B.Cu" "B.Mask" "B.Paste")
 			(roundrect_rratio 0.25)
-			(net "ROW1_R")
+			(net "ROW2_R")
 			(pinfunction "K_1")
 			(pintype "passive")
@@
 			(layers "B.Cu" "B.Mask" "B.Paste")
 			(roundrect_rratio 0.25)
-			(net "ROW0")
+			(net "ROW2")
 			(pinfunction "K_1")
 			(pintype "passive")
@@
 			(layers "B.Cu" "B.Mask" "B.Paste")
 			(roundrect_rratio 0.25)
-			(net "ROW1")
+			(net "ROW0")
 			(pinfunction "K_1")
 			(pintype "passive")
@@
 			(layers "B.Cu" "B.Mask" "B.Paste")
 			(roundrect_rratio 0.25)
-			(net "ROW0_R")
+			(net "ROW1_R")
 			(pinfunction "K_1")
 			(pintype "passive")
@@
 			(layers "B.Cu" "B.Mask" "B.Paste")
 			(roundrect_rratio 0.25)
-			(net "ROW0")
+			(net "ROW1")
 			(pinfunction "K_1")
 			(pintype "passive")
@@
 			(layers "B.Cu" "B.Mask" "B.Paste")
 			(roundrect_rratio 0.25)
-			(net "ROW1")
+			(net "ROW2")
 			(pinfunction "K_1")
 			(pintype "passive")
@@
 			(layers "B.Cu" "B.Mask" "B.Paste")
 			(roundrect_rratio 0.25)
-			(net "ROW3_R")
+			(net "ROW2_R")
 			(pinfunction "K_1")
 			(pintype "passive")

Commit message: feat: added routing to the left pcb
Parts:
- added MH10_R1: MountingHole_2.2mm_M2, MountingHole:MountingHole_2.2mm_M2, F.Cu at (239.1, 158.3)
- added MH3: MountingHole_2.2mm_M2, MountingHole:MountingHole_2.2mm_M2, F.Cu at (124.8, 105.5)
- added MH4: MountingHole_2.2mm_M2, MountingHole:MountingHole_2.2mm_M2, F.Cu at (140.8, 147.9)
- added MH7_R1: MountingHole_2.2mm_M2, MountingHole:MountingHole_2.2mm_M2, F.Cu at (294.6, 105.5)
- moved MH8_R1 22.5 mm to (278.4, 147.9)
- moved MH6 19.0 mm to (180.7, 158.3)
- moved R713_R1 7.75 mm to (233.0, 117.0), turned to 0 degrees
- moved R715_R1 2.36 mm to (220.9, 119.3)
- moved R714_R1 2.24 mm to (218.8, 119.3)
- moved R9 0.41 mm to (109.5, 114.6)
- moved BT1 0.35 mm to (190.1, 156.5)
- moved MH1 0.26 mm to (85.8, 115.0)
- moved D47_R1 0.23 mm to (335.8, 101.1)
- moved D48_R1 0.23 mm to (340.7, 101.1)
- moved D50_R1 0.23 mm to (345.6, 101.1)
- moved D52_R1 0.23 mm to (350.4, 101.1)
- turned D46 to -29 degrees
- turned F1 to 0 degrees
- renumbered MH3 to MH5, MH4 to MH6, MH7_R1 to MH9_R1
Routing:
- net VBAT: track 0.00 -> 573.7 mm, vias 0 -> 3
- net Net-(D21-VDD): track 0.00 -> 223.6 mm, vias 0 -> 4
- net COL1: track 0.00 -> 193.2 mm, vias 0 -> 4
- net Net-(D21-DIN): track 0.00 -> 170.6 mm, vias 0 -> 2
- net COL0: track 0.00 -> 168.2 mm, vias 0 -> 6
- net COL3: track 0.00 -> 144.9 mm, vias 0 -> 4
- net COL4: track 0.00 -> 139.7 mm, vias 0 -> 9
- net COL2: track 0.00 -> 126.7 mm, vias 0 -> 8
- net BL_DRAIN: track 0.00 -> 121.2 mm, vias 0 -> 8
- net VBAT_R: track 0.00 -> 119.0 mm, vias 0 -> 2
- net ROW0: track 0.00 -> 118.8 mm, vias 0 -> 12
- net COL5: track 0.00 -> 107.6 mm, vias 0 -> 2
- net ROW2: track 0.00 -> 89.6 mm, vias 0 -> 6
- net VBAT_RAW_R: track 0.00 -> 69.2 mm
- net VBAT_RAW: track 0.00 -> 68.5 mm, vias 0 -> 2
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