File: keyboard/kicad/revisions/dormin-rev_1.0/dormin.kicad_pcb (KiCad board)
At the start: 2 copper layers, 288.7 x 103.4 mm, 234 parts, among them J1 Conn_01x06, J2 Conn_01x04, J3 Conn_01x02, J4_R1 Conn_01x06, J4_R2 Conn_01x02, J6_R1 Conn_01x04, Q1 AO3400A, Q2 AO3407A, Q3_R1 AO3407A, Q4_R1 AO3400A, SW1 SW_Push, SW10 SW_Push, SW11 SW_Push, SW12 SW_Push, SW13 SW_Push, SW14 SW_Push, SW15 SW_Push, SW16 SW_Push, SW17 SW_Push, SW18 SW_Push, SW19 SW_Push, SW2 SW_Push, SW20 SW_Push, SW21 SW_Push, SW22 SW_Push, SW23 SW_Push, SW24 SW_Push, SW25 SW_Push, SW26 SW_Push, SW27 SW_Push, SW28 SW_Push, SW29 SW_Push, SW3 SW_Push, SW30 SW_Push, SW31 SW_Push, SW32 SW_Push, SW33 SW_Push, SW34 SW_Push, SW35 SW_Push, SW36 SW_Push, SW37 SW_Push, SW38 SW_Push, SW39 SW_Push, SW4 SW_Push, SW40 SW_Push, SW5 SW_Push, SW6 SW_Push, SW7 SW_Push, SW8 SW_Push, SW9 SW_Push, U3 XIAO-nRF52840-Plus-SMD, U5_R1 XIAO-nRF52840-Plus-SMD

Commit message: feat: improved ergogen config and exported pcb
Parts:
- removed BT1, BT2_R1: Pads, willkeebs_power:Battery_Pad
- removed C1, C3, C5_R1, C7_R1: 10uF, Capacitor_SMD:C_0603_1608Metric
- removed C2, C4, C6_R1, C8_R1: 100nF, Capacitor_SMD:C_0603_1608Metric
- removed D1, D10, D11, D12, D13, D14, D15, D16, D17, D18, D19, D2, D20, D3, D4, D5, D6, D61_R1, D62_R1, D63_R1, D64_R1, D7, D72_R1, D73_R1, D74_R1, D75_R1, D8, D81_R1, D82_R1, D83_R1, D84_R1, D85_R1, D86_R1, D87_R1, D88_R1, D89_R1, D9, D90_R1, D91_R1, D92_R1: 1N4148W, Diode_SMD:D_SOD-123
- removed D21, D22, D23, D24, D47_R1, D48_R1, D50_R1, D52_R1: SK6812MINI-E, LED_SMD:LED_SK6812MINI-E_3.2x2.8mm_P1.5mm_ReverseMount
- removed D25, D26, D29, D30, D31, D32, D33, D34, D35, D36, D37, D38, D39, D40, D41, D42, D43, D44, D45, D46, D53_R1, D54_R1, D55_R1, D56_R1, D57_R1, D58_R1, D59_R1, D60_R1, D65_R1, D66_R1, D67_R1, D68_R1, D69_R1, D70_R1, D71_R1, D76_R1, D77_R1, D78_R1, D79_R1, D80_R1: LED, willkeebs_components:LED_MHT151WDT
- removed D27, D47_R2: D_Schottky, Diode_SMD:D_SOD-523
- removed D28, D48_R2: KPESD5V0S1UL, Diode_SMD:D_SOD-882
- removed F1, F2_R1: Polyfuse, Fuse:Fuse_1206_3216Metric
- removed J1, J4_R1: Conn_01x06, willkeebs_misc:SMD_Conn_1x06_P2.54mm_Vertical
- removed J2, J6_R1: Conn_01x04, Connector_PinSocket_2.54mm:PinSocket_1x04_P2.54mm_Vertical
- removed J3, J4_R2: Conn_01x02, willkeebs_misc:SMD_Conn_1x02_P2.54mm_Vertical
- removed JST1, JST2_R1: Conn_01x02_Pin, Connector_JST:JST_GH_SM02B-GHS-TB_1x02-1MP_P1.25mm_Horizontal
- removed MH1, MH10_R1, MH2, MH3, MH4, MH5, MH5_R1, MH6, MH6_R1, MH7_R1, MH8_R1, MH9_R1: MountingHole_2.2mm_M2, MountingHole:MountingHole_2.2mm_M2
- removed PSW1, PSW2_R1: SW_SPDT, PCM_marbastlib-various:SW_MSK12C02-HB
- removed Q1, Q4_R1: AO3400A, Package_TO_SOT_SMD:SOT-23
- removed Q2, Q3_R1: AO3407A, Package_TO_SOT_SMD:SOT-23
- removed R1, R10, R11, R12, R13, R14, R15, R16, R17, R18, R19, R2, R20, R21, R22, R25_R1, R26_R1, R27_R1, R28_R1, R29_R1, R3, R30_R1, R31_R1, R32_R1, R33_R1, R34_R1, R35_R1, R36_R1, R37_R1, R38_R1, R39_R1, R4, R40_R1, R41_R1, R42_R1, R43_R1, R44_R1, R7, R8, R9: 1K, Resistor_SMD:R_0603_1608Metric
- removed R706, R708_R1, R710, R713_R1: 100R, Resistor_SMD:R_0603_1608Metric
- removed R707, R709_R1: 10k, Resistor_SMD:R_0603_1608Metric
- removed R711, R714_R1: 100k, Resistor_SMD:R_0603_1608Metric
- removed R712, R715_R1: 330R, Resistor_SMD:R_0603_1608Metric
- removed REF** (x4): BreakLine_5h_D0.5mm_P0.85mm, Panelization:BreakLine_5h_D0.5mm_P0.85mm
- removed RSW1, RSW2_R1: RSW1, Button_Switch_SMD:SW_SPST_SKQG_WithStem
- removed TP1: VBAT, TestPoint:TestPoint_Pad_D1.0mm
- removed TP2, TP5_R1: GND, TestPoint:TestPoint_Pad_D1.0mm
- removed TP3: STS_LED_EN, TestPoint:TestPoint_Pad_D1.0mm
- removed TP4_R1: VBAT_R, TestPoint:TestPoint_Pad_D1.0mm
- removed TP6_R1: STS_LED_EN_R, TestPoint:TestPoint_Pad_D1.0mm
- removed U3, U5_R1: XIAO-nRF52840-Plus-SMD, Seeed_Studio_XIAO_Series:XIAO-nRF52840-Plus-SMD
- SW1, SW10, SW11, SW12, SW13, SW14, SW15, SW16, SW17, SW18, SW19, SW2, SW20, SW21, SW22, SW23, SW24, SW25, SW26, SW27, SW28, SW29, SW3, SW30, SW31, SW32, SW33, SW34, SW35, SW36, SW37, SW38, SW39, SW4, SW40, SW5, SW6, SW7, SW8, SW9: footprint willkeebs_keyboard:NF_LED_1206_SW_KS33_3_0_HS_1U -> SW_MX_Choc_Hotswap
- moved SW24 8.93 mm to (330.0, 131.0), turned to 0 degrees
- moved SW36 8.93 mm to (253.8, 131.0), turned to 0 degrees
- moved SW21 8.93 mm to (349.1, 140.5), turned to 0 degrees
- moved SW22 8.93 mm to (349.1, 121.4), turned to 0 degrees
- moved SW23 8.93 mm to (330.0, 150.0), turned to 0 degrees
- moved SW25 8.93 mm to (330.0, 111.9), turned to 0 degrees
- moved SW26 8.93 mm to (311.0, 145.2), turned to 0 degrees
- moved SW27 8.93 mm to (311.0, 126.2), turned to 0 degrees
- moved SW28 8.93 mm to (311.0, 107.1), turned to 0 degrees
- moved SW29 8.93 mm to (291.9, 140.5), turned to 0 degrees
- moved SW30 8.93 mm to (291.9, 121.4), turned to 0 degrees
- moved SW31 8.93 mm to (291.9, 102.4), turned to 0 degrees
- moved SW32 8.93 mm to (272.9, 145.2), turned to 0 degrees
- moved SW33 8.93 mm to (272.9, 126.2), turned to 0 degrees
- moved SW34 8.93 mm to (272.9, 107.1), turned to 0 degrees
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Connections:
- SW1 pad 1: Net-(D1-A) -> outer_home_from
- SW1 pad 2: COL0 -> outer_home_to
- SW10 pad 1: Net-(D10-A) -> middle_home_from
- SW10 pad 2: COL3 -> middle_home_to
- SW11 pad 1: Net-(D11-A) -> middle_top_from
- SW11 pad 2: COL3 -> middle_top_to
- SW12 pad 1: Net-(D12-A) -> index_bottom_from
- SW12 pad 2: COL4 -> index_bottom_to
- SW13 pad 1: Net-(D13-A) -> index_home_from
- SW13 pad 2: COL4 -> index_home_to
- SW14 pad 1: Net-(D14-A) -> index_top_from
- SW14 pad 2: COL4 -> index_top_to
- SW15 pad 1: Net-(D15-A) -> inner_bottom_from
- SW15 pad 2: COL5 -> inner_bottom_to
- SW16 pad 1: Net-(D16-A) -> inner_home_from
- SW16 pad 2: COL5 -> inner_home_to
- SW17 pad 1: Net-(D17-A) -> inner_top_from
- SW17 pad 2: COL5 -> inner_top_to
- SW18 pad 1: Net-(D18-A) -> inner_only_from
- SW18 pad 2: COL3 -> inner_only_to
- SW19 pad 1: Net-(D19-A) -> home_only_from
- SW19 pad 2: COL4 -> home_only_to
- SW2 pad 1: Net-(D2-A) -> outer_top_from
- SW2 pad 2: COL0 -> outer_top_to
- SW20 pad 1: Net-(D20-A) -> outer_only_from
- SW20 pad 2: COL5 -> outer_only_to
- SW21 pad 1: Net-(D61_R1-A) -> mirror_outer_home_from
- SW21 pad 2: COL5_R -> mirror_outer_home_to
- SW22 pad 1: Net-(D62_R1-A) -> mirror_outer_top_from
- SW22 pad 2: COL5_R -> mirror_outer_top_to
- SW23 pad 1: Net-(D63_R1-A) -> mirror_pinky_bottom_from
- SW23 pad 2: COL4_R -> mirror_pinky_bottom_to
- SW24 pad 1: Net-(D64_R1-A) -> mirror_pinky_home_from
- SW24 pad 2: COL4_R -> mirror_pinky_home_to
- SW25 pad 1: Net-(D72_R1-A) -> mirror_pinky_top_from
- SW25 pad 2: COL4_R -> mirror_pinky_top_to
- SW26 pad 1: Net-(D73_R1-A) -> mirror_ring_bottom_from
- SW26 pad 2: COL3_R -> mirror_ring_bottom_to
- SW27 pad 1: Net-(D74_R1-A) -> mirror_ring_home_from
- SW27 pad 2: COL3_R -> mirror_ring_home_to
- SW28 pad 1: Net-(D75_R1-A) -> mirror_ring_top_from
- SW28 pad 2: COL3_R -> mirror_ring_top_to
- SW29 pad 1: Net-(D81_R1-A) -> mirror_middle_bottom_from
- SW29 pad 2: COL2_R -> mirror_middle_bottom_to
- SW3 pad 1: Net-(D3-A) -> pinky_bottom_from
- SW3 pad 2: COL1 -> pinky_bottom_to
- SW30 pad 1: Net-(D82_R1-A) -> mirror_middle_home_from
- SW30 pad 2: COL2_R -> mirror_middle_home_to
- SW31 pad 1: Net-(D83_R1-A) -> mirror_middle_top_from
- SW31 pad 2: COL2_R -> mirror_middle_top_to
- SW32 pad 1: Net-(D84_R1-A) -> mirror_index_bottom_from
- SW32 pad 2: COL1_R -> mirror_index_bottom_to
- SW33 pad 1: Net-(D85_R1-A) -> mirror_index_home_from
- SW33 pad 2: COL1_R -> mirror_index_home_to
- SW34 pad 1: Net-(D86_R1-A) -> mirror_index_top_from
- SW34 pad 2: COL1_R -> mirror_index_top_to
- SW35 pad 1: Net-(D87_R1-A) -> mirror_inner_bottom_from
- SW35 pad 2: COL0_R -> mirror_inner_bottom_to
- SW36 pad 1: Net-(D88_R1-A) -> mirror_inner_home_from
- SW36 pad 2: COL0_R -> mirror_inner_home_to
- SW37 pad 1: Net-(D89_R1-A) -> mirror_inner_top_from
- SW37 pad 2: COL0_R -> mirror_inner_top_to
- SW38 pad 1: Net-(D90_R1-A) -> mirror_inner_only_from
- SW38 pad 2: COL0_R -> mirror_inner_only_to
- SW39 pad 1: Net-(D91_R1-A) -> mirror_home_only_from
- SW39 pad 2: COL1_R -> mirror_home_only_to
- SW4 pad 1: Net-(D4-A) -> pinky_home_from
- SW4 pad 2: COL1 -> pinky_home_to
- SW40 pad 1: Net-(D92_R1-A) -> mirror_outer_only_from
- SW40 pad 2: COL2_R -> mirror_outer_only_to
- SW5 pad 1: Net-(D5-A) -> pinky_top_from
- SW5 pad 2: COL1 -> pinky_top_to
- SW6 pad 1: Net-(D6-A) -> ring_bottom_from
- SW6 pad 2: COL2 -> ring_bottom_to
- SW7 pad 1: Net-(D7-A) -> ring_home_from
- SW7 pad 2: COL2 -> ring_home_to
- SW8 pad 1: Net-(D8-A) -> ring_top_from
- SW8 pad 2: COL2 -> ring_top_to
- SW9 pad 1: Net-(D9-A) -> middle_bottom_from
- SW9 pad 2: COL3 -> middle_bottom_to
Routing:
- net VBAT: track 573.7 -> 0.00 mm, vias 3 -> 0
- net Net-(D21-VDD): track 223.6 -> 0.00 mm, vias 4 -> 0
- net COL1: track 193.2 -> 0.00 mm, vias 4 -> 0
- net Net-(D21-DIN): track 170.6 -> 0.00 mm, vias 2 -> 0
- net COL0: track 168.2 -> 0.00 mm, vias 6 -> 0
- net COL3: track 144.9 -> 0.00 mm, vias 4 -> 0
- net COL4: track 139.7 -> 0.00 mm, vias 9 -> 0
- net COL2: track 126.7 -> 0.00 mm, vias 8 -> 0
- net BL_DRAIN: track 121.2 -> 0.00 mm, vias 8 -> 0
- net VBAT_R: track 119.0 -> 0.00 mm, vias 2 -> 0
- net ROW0: track 118.8 -> 0.00 mm, vias 12 -> 0
- net COL5: track 107.6 -> 0.00 mm, vias 2 -> 0
- net ROW2: track 89.6 -> 0.00 mm, vias 6 -> 0
- net VBAT_RAW_R: track 69.2 -> 0.00 mm
- net VBAT_RAW: track 68.5 -> 0.00 mm, vias 2 -> 0
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Other:
- board size 288.7 x 103.4 mm -> 289.7 x 102.8 mm
- board text removed: "3V3"
- board text removed: "EXTA"
- board text removed: "EXTB"
- board text removed: "GND"
- board text removed: "SCL"
- board text removed: "SDA"
- board text removed: "SWC"
- board text removed: "SWD"

Commit message: feat: added new pcb design
Parts:
- added BT1: Pads, willkeebs_power:Battery_Pad, F.Cu at (-19.7, 209.3)
- added BT2_R1: Pads, willkeebs_power:Battery_Pad, F.Cu at (-19.7, 263.2)
- added C1: 10uF, Capacitor_SMD:C_0603_1608Metric, F.Cu at (-67.8, 199.8)
- added C2: 100nF, Capacitor_SMD:C_0603_1608Metric, F.Cu at (-67.8, 202.4)
- added C3: 10uF, Capacitor_SMD:C_0603_1608Metric, F.Cu at (-67.8, 204.9)
- added C4: 100nF, Capacitor_SMD:C_0603_1608Metric, F.Cu at (-67.8, 207.4)
- added C5_R1: 10uF, Capacitor_SMD:C_0603_1608Metric, F.Cu at (-67.8, 253.7)
- added C6_R1: 100nF, Capacitor_SMD:C_0603_1608Metric, F.Cu at (-67.8, 256.2)
- added C7_R1: 10uF, Capacitor_SMD:C_0603_1608Metric, F.Cu at (-67.8, 258.7)
- added C8_R1: 100nF, Capacitor_SMD:C_0603_1608Metric, F.Cu at (-67.8, 261.2)
- added D1: 1N4148W, Diode_SMD:D_SOD-123, F.Cu at (-44.2, 197.5)
- added D10: 1N4148W, Diode_SMD:D_SOD-123, F.Cu at (-38.5, 210.9)
- added D11: 1N4148W, Diode_SMD:D_SOD-123, F.Cu at (-32.7, 197.5)
- added D12: 1N4148W, Diode_SMD:D_SOD-123, F.Cu at (-32.7, 200.9)
- added D13: 1N4148W, Diode_SMD:D_SOD-123, F.Cu at (-32.7, 204.2)
- added D14: 1N4148W, Diode_SMD:D_SOD-123, F.Cu at (-32.7, 207.6)
- added D15: 1N4148W, Diode_SMD:D_SOD-123, F.Cu at (-32.7, 210.9)
- added D16: 1N4148W, Diode_SMD:D_SOD-123, F.Cu at (-26.9, 197.5)
- added D17: 1N4148W, Diode_SMD:D_SOD-123, F.Cu at (-26.9, 200.9)
- added D18: 1N4148W, Diode_SMD:D_SOD-123, F.Cu at (-26.9, 204.2)
- added D19: 1N4148W, Diode_SMD:D_SOD-123, F.Cu at (-26.9, 207.6)
- added D2: 1N4148W, Diode_SMD:D_SOD-123, F.Cu at (-44.2, 200.9)
- added D20: 1N4148W, Diode_SMD:D_SOD-123, F.Cu at (-26.9, 210.9)
- added D21: SK6812MINI-E, LED_SMD:LED_SK6812MINI-E_3.2x2.8mm_P1.5mm_ReverseMount, B.Cu at (73.3, 108.0)
- added D22: SK6812MINI-E, LED_SMD:LED_SK6812MINI-E_3.2x2.8mm_P1.5mm_ReverseMount, B.Cu at (78.4, 108.0)
- added D23: SK6812MINI-E, LED_SMD:LED_SK6812MINI-E_3.2x2.8mm_P1.5mm_ReverseMount, B.Cu at (83.4, 108.0)
- added D24: SK6812MINI-E, LED_SMD:LED_SK6812MINI-E_3.2x2.8mm_P1.5mm_ReverseMount, B.Cu at (88.5, 108.0)
- added D25: LED, willkeebs_components:LED_MHT151WDT, F.Cu at (-67.0, 178.5)
- added D26: LED, willkeebs_components:LED_MHT151WDT, F.Cu at (-67.0, 183.0)
- added D27: D_Schottky, Diode_SMD:D_SOD-523, F.Cu at (-39.7, 225.7)
- added D28: KPESD5V0S1UL, Diode_SMD:D_SOD-882, F.Cu at (-36.6, 225.7)
- added D29: LED, willkeebs_components:LED_MHT151WDT, F.Cu at (-67.0, 187.5)
- added D3: 1N4148W, Diode_SMD:D_SOD-123, F.Cu at (-44.2, 204.2)
- added D30: LED, willkeebs_components:LED_MHT151WDT, F.Cu at (-67.0, 192.1)
- added D31: LED, willkeebs_components:LED_MHT151WDT, F.Cu at (-67.0, 196.6)
- added D32: LED, willkeebs_components:LED_MHT151WDT, F.Cu at (-61.3, 178.5)
- added D33: LED, willkeebs_components:LED_MHT151WDT, F.Cu at (-61.3, 183.0)
- added D34: LED, willkeebs_components:LED_MHT151WDT, F.Cu at (-61.3, 187.5)
- added D35: LED, willkeebs_components:LED_MHT151WDT, F.Cu at (-61.3, 192.1)
- added D36: LED, willkeebs_components:LED_MHT151WDT, F.Cu at (-61.3, 196.6)
- added D37: LED, willkeebs_components:LED_MHT151WDT, F.Cu at (-55.7, 178.5)
- added D38: LED, willkeebs_components:LED_MHT151WDT, F.Cu at (-55.7, 183.0)
- added D39: LED, willkeebs_components:LED_MHT151WDT, F.Cu at (-55.7, 187.5)
- added D4: 1N4148W, Diode_SMD:D_SOD-123, F.Cu at (-44.2, 207.6)
- added D40: LED, willkeebs_components:LED_MHT151WDT, F.Cu at (-55.7, 192.1)
- added D41: LED, willkeebs_components:LED_MHT151WDT, F.Cu at (-55.7, 196.6)
- added D42: LED, willkeebs_components:LED_MHT151WDT, F.Cu at (-50.0, 178.5)
- added D43: LED, willkeebs_components:LED_MHT151WDT, F.Cu at (-50.0, 183.0)
- added D44: LED, willkeebs_components:LED_MHT151WDT, F.Cu at (-50.0, 187.5)
- added D45: LED, willkeebs_components:LED_MHT151WDT, F.Cu at (-50.0, 192.1)
- added D46: LED, willkeebs_components:LED_MHT151WDT, F.Cu at (-50.0, 196.6)
- added D47_R1: SK6812MINI-E, LED_SMD:LED_SK6812MINI-E_3.2x2.8mm_P1.5mm_ReverseMount, B.Cu at (356.8, 108.0)
- added D47_R2: D_Schottky, Diode_SMD:D_SOD-523, F.Cu at (-39.7, 279.6)
- added D48_R1: SK6812MINI-E, LED_SMD:LED_SK6812MINI-E_3.2x2.8mm_P1.5mm_ReverseMount, B.Cu at (351.7, 108.0)
- added D48_R2: KPESD5V0S1UL, Diode_SMD:D_SOD-882, F.Cu at (-36.6, 279.5)
- added D5: 1N4148W, Diode_SMD:D_SOD-123, F.Cu at (-44.2, 210.9)
- added D50_R1: SK6812MINI-E, LED_SMD:LED_SK6812MINI-E_3.2x2.8mm_P1.5mm_ReverseMount, B.Cu at (346.7, 108.0)
- added D52_R1: SK6812MINI-E, LED_SMD:LED_SK6812MINI-E_3.2x2.8mm_P1.5mm_ReverseMount, B.Cu at (341.7, 108.0)
- added D53_R1: LED, willkeebs_components:LED_MHT151WDT, F.Cu at (-67.0, 232.3)
- added D54_R1: LED, willkeebs_components:LED_MHT151WDT, F.Cu at (-67.0, 236.9)
- added D55_R1: LED, willkeebs_components:LED_MHT151WDT, F.Cu at (-67.0, 241.4)
- added D56_R1: LED, willkeebs_components:LED_MHT151WDT, F.Cu at (-67.0, 245.9)
- added D57_R1: LED, willkeebs_components:LED_MHT151WDT, F.Cu at (-67.0, 250.4)
- added D58_R1: LED, willkeebs_components:LED_MHT151WDT, F.Cu at (-61.3, 232.3)
- added D59_R1: LED, willkeebs_components:LED_MHT151WDT, F.Cu at (-61.3, 236.9)
- added D6: 1N4148W, Diode_SMD:D_SOD-123, F.Cu at (-38.5, 197.5)
- added D60_R1: LED, willkeebs_components:LED_MHT151WDT, F.Cu at (-61.3, 241.4)
- added D61_R1: 1N4148W, Diode_SMD:D_SOD-123, F.Cu at (-44.2, 251.4)
- added D62_R1: 1N4148W, Diode_SMD:D_SOD-123, F.Cu at (-44.2, 254.7)
- added D63_R1: 1N4148W, Diode_SMD:D_SOD-123, F.Cu at (-44.2, 258.1)
- added D64_R1: 1N4148W, Diode_SMD:D_SOD-123, F.Cu at (-44.2, 261.4)
- added D65_R1: LED, willkeebs_components:LED_MHT151WDT, F.Cu at (-61.3, 245.9)
- added D66_R1: LED, willkeebs_components:LED_MHT151WDT, F.Cu at (-61.3, 250.4)
- added D67_R1: LED, willkeebs_components:LED_MHT151WDT, F.Cu at (-55.7, 232.3)
- added D68_R1: LED, willkeebs_components:LED_MHT151WDT, F.Cu at (-55.7, 236.9)
- added D69_R1: LED, willkeebs_components:LED_MHT151WDT, F.Cu at (-55.7, 241.4)
- added D7: 1N4148W, Diode_SMD:D_SOD-123, F.Cu at (-38.5, 200.9)
- added D70_R1: LED, willkeebs_components:LED_MHT151WDT, F.Cu at (-55.7, 245.9)
- added D71_R1: LED, willkeebs_components:LED_MHT151WDT, F.Cu at (-55.7, 250.4)
- added D72_R1: 1N4148W, Diode_SMD:D_SOD-123, F.Cu at (-44.2, 264.8)
- added D73_R1: 1N4148W, Diode_SMD:D_SOD-123, F.Cu at (-38.5, 251.4)
- added D74_R1: 1N4148W, Diode_SMD:D_SOD-123, F.Cu at (-38.5, 254.7)
- added D75_R1: 1N4148W, Diode_SMD:D_SOD-123, F.Cu at (-38.5, 258.1)
- added D76_R1: LED, willkeebs_components:LED_MHT151WDT, F.Cu at (-50.0, 232.3)
- added D77_R1: LED, willkeebs_components:LED_MHT151WDT, F.Cu at (-50.0, 236.9)
- added D78_R1: LED, willkeebs_components:LED_MHT151WDT, F.Cu at (-50.0, 241.4)
- added D79_R1: LED, willkeebs_components:LED_MHT151WDT, F.Cu at (-50.0, 245.9)
- added D8: 1N4148W, Diode_SMD:D_SOD-123, F.Cu at (-38.5, 204.2)
- added D80_R1: LED, willkeebs_components:LED_MHT151WDT, F.Cu at (-50.0, 250.4)
- added D81_R1: 1N4148W, Diode_SMD:D_SOD-123, F.Cu at (-38.5, 261.4)
- added D82_R1: 1N4148W, Diode_SMD:D_SOD-123, F.Cu at (-38.5, 264.8)
- added D83_R1: 1N4148W, Diode_SMD:D_SOD-123, F.Cu at (-32.7, 251.4)
- added D84_R1: 1N4148W, Diode_SMD:D_SOD-123, F.Cu at (-32.7, 254.7)
- added D85_R1: 1N4148W, Diode_SMD:D_SOD-123, F.Cu at (-32.7, 258.1)
- added D86_R1: 1N4148W, Diode_SMD:D_SOD-123, F.Cu at (-32.7, 261.4)
- added D87_R1: 1N4148W, Diode_SMD:D_SOD-123, F.Cu at (-32.7, 264.8)
- added D88_R1: 1N4148W, Diode_SMD:D_SOD-123, F.Cu at (-26.9, 251.4)
- added D89_R1: 1N4148W, Diode_SMD:D_SOD-123, F.Cu at (-26.9, 254.7)
- added D9: 1N4148W, Diode_SMD:D_SOD-123, F.Cu at (-38.5, 207.6)
- added D90_R1: 1N4148W, Diode_SMD:D_SOD-123, F.Cu at (-26.9, 258.1)
- added D91_R1: 1N4148W, Diode_SMD:D_SOD-123, F.Cu at (-26.9, 261.4)
- added D92_R1: 1N4148W, Diode_SMD:D_SOD-123, F.Cu at (-26.9, 264.8)
- added F1: Polyfuse, Fuse:Fuse_1206_3216Metric, F.Cu at (-44.4, 226.2)
- added F2_R1: Polyfuse, Fuse:Fuse_1206_3216Metric, F.Cu at (-44.4, 280.0)
- added J1: Conn_01x06, willkeebs_misc:SMD_Conn_1x06_P2.54mm_Vertical, F.Cu at (-50.1, 200.9)
- added J2: Conn_01x04, Connector_PinSocket_2.54mm:PinSocket_1x04_P2.54mm_Vertical, F.Cu at (-21.7, 198.1)
- added J3: Conn_01x02, willkeebs_components:Pogo1x2-Right-Angle, B.Cu at (207.5, 140.0)
- added J4_R1: Conn_01x06, willkeebs_misc:SMD_Conn_1x06_P2.54mm_Vertical, F.Cu at (-50.1, 254.7)
- added J4_R2: Conn_01x02, willkeebs_components:Pogo1x2-Right-Angle, B.Cu at (222.6, 140.0)
- added J6_R1: Conn_01x04, Connector_PinSocket_2.54mm:PinSocket_1x04_P2.54mm_Vertical, F.Cu at (-21.7, 252.0)
- added JST1: Conn_01x02_Pin, Connector_JST:JST_GH_SM02B-GHS-TB_1x02-1MP_P1.25mm_Horizontal, F.Cu at (-65.8, 222.4)
- added JST2_R1: Conn_01x02_Pin, Connector_JST:JST_GH_SM02B-GHS-TB_1x02-1MP_P1.25mm_Horizontal, F.Cu at (-65.8, 276.2)
- added MH1: MountingHole_2.2mm_M2, MountingHole:MountingHole_2.2mm_M2, F.Cu at (-44.2, 215.6)
- added MH10_R1: MountingHole_2.2mm_M2, MountingHole:MountingHole_2.2mm_M2, F.Cu at (-44.2, 269.4)
- added MH2: MountingHole_2.2mm_M2, MountingHole:MountingHole_2.2mm_M2, F.Cu at (-44.2, 221.5)
- added MH3: MountingHole_2.2mm_M2, MountingHole:MountingHole_2.2mm_M2, F.Cu at (-38.2, 215.6)
- added MH4: MountingHole_2.2mm_M2, MountingHole:MountingHole_2.2mm_M2, F.Cu at (-38.2, 221.5)
- added MH5: MountingHole_2.2mm_M2, MountingHole:MountingHole_2.2mm_M2, F.Cu at (-32.3, 215.6)
- added MH5_R1: MountingHole_2.2mm_M2, MountingHole:MountingHole_2.2mm_M2, F.Cu at (-44.2, 275.4)
- added MH6: MountingHole_2.2mm_M2, MountingHole:MountingHole_2.2mm_M2, F.Cu at (-32.3, 221.5)
- added MH6_R1: MountingHole_2.2mm_M2, MountingHole:MountingHole_2.2mm_M2, F.Cu at (-38.2, 269.4)
- added MH7_R1: MountingHole_2.2mm_M2, MountingHole:MountingHole_2.2mm_M2, F.Cu at (-38.2, 275.4)
- added MH8_R1: MountingHole_2.2mm_M2, MountingHole:MountingHole_2.2mm_M2, F.Cu at (-32.3, 269.4)
- added MH9_R1: MountingHole_2.2mm_M2, MountingHole:MountingHole_2.2mm_M2, F.Cu at (-32.3, 275.4)
- added PSW1: SW_SPDT, PCM_marbastlib-various:SW_MSK12C02-HB, B.Cu at (187.3, 102.7)
- added PSW2_R1: SW_SPDT, PCM_marbastlib-various:SW_MSK12C02-HB, B.Cu at (243.0, 102.7)
- added Q1: AO3400A, Package_TO_SOT_SMD:SOT-23, F.Cu at (-59.3, 220.9)
- added Q2: AO3407A, Package_TO_SOT_SMD:SOT-23, F.Cu at (-59.3, 225.3)
- added Q3_R1: AO3407A, Package_TO_SOT_SMD:SOT-23, F.Cu at (-59.3, 274.7)
- added Q4_R1: AO3400A, Package_TO_SOT_SMD:SOT-23, F.Cu at (-59.3, 279.2)
- added R1: 1K, Resistor_SMD:R_0603_1608Metric, F.Cu at (-67.8, 209.9)
- added R10: 1K, Resistor_SMD:R_0603_1608Metric, F.Cu at (-63.8, 207.4)
- added R11: 1K, Resistor_SMD:R_0603_1608Metric, F.Cu at (-63.8, 209.9)
- added R12: 1K, Resistor_SMD:R_0603_1608Metric, F.Cu at (-63.8, 212.4)
- added R13: 1K, Resistor_SMD:R_0603_1608Metric, F.Cu at (-63.8, 214.9)
- added R14: 1K, Resistor_SMD:R_0603_1608Metric, F.Cu at (-63.8, 217.4)
- added R15: 1K, Resistor_SMD:R_0603_1608Metric, F.Cu at (-59.8, 199.8)
- added R16: 1K, Resistor_SMD:R_0603_1608Metric, F.Cu at (-59.8, 202.4)
- added R17: 1K, Resistor_SMD:R_0603_1608Metric, F.Cu at (-59.8, 204.9)
- added R18: 1K, Resistor_SMD:R_0603_1608Metric, F.Cu at (-59.8, 207.4)
- added R19: 1K, Resistor_SMD:R_0603_1608Metric, F.Cu at (-59.8, 209.9)
- added R2: 1K, Resistor_SMD:R_0603_1608Metric, F.Cu at (-67.8, 212.4)
- added R20: 1K, Resistor_SMD:R_0603_1608Metric, F.Cu at (-59.8, 212.4)
- added R21: 1K, Resistor_SMD:R_0603_1608Metric, F.Cu at (-59.8, 214.9)
- added R22: 1K, Resistor_SMD:R_0603_1608Metric, F.Cu at (-59.8, 217.4)
- added R25_R1: 1K, Resistor_SMD:R_0603_1608Metric, F.Cu at (-67.8, 263.7)
- added R26_R1: 1K, Resistor_SMD:R_0603_1608Metric, F.Cu at (-67.8, 266.2)
- added R27_R1: 1K, Resistor_SMD:R_0603_1608Metric, F.Cu at (-67.8, 268.7)
- added R28_R1: 1K, Resistor_SMD:R_0603_1608Metric, F.Cu at (-67.8, 271.2)
- added R29_R1: 1K, Resistor_SMD:R_0603_1608Metric, F.Cu at (-63.8, 253.7)
- added R3: 1K, Resistor_SMD:R_0603_1608Metric, F.Cu at (-67.8, 214.9)
- added R30_R1: 1K, Resistor_SMD:R_0603_1608Metric, F.Cu at (-63.8, 256.2)
- added R31_R1: 1K, Resistor_SMD:R_0603_1608Metric, F.Cu at (-63.8, 258.7)
- added R32_R1: 1K, Resistor_SMD:R_0603_1608Metric, F.Cu at (-63.8, 261.2)
- added R33_R1: 1K, Resistor_SMD:R_0603_1608Metric, F.Cu at (-63.8, 263.7)
- added R34_R1: 1K, Resistor_SMD:R_0603_1608Metric, F.Cu at (-63.8, 266.2)
- added R35_R1: 1K, Resistor_SMD:R_0603_1608Metric, F.Cu at (-63.8, 268.7)
- added R36_R1: 1K, Resistor_SMD:R_0603_1608Metric, F.Cu at (-63.8, 271.2)
- added R37_R1: 1K, Resistor_SMD:R_0603_1608Metric, F.Cu at (-59.8, 253.7)
- added R38_R1: 1K, Resistor_SMD:R_0603_1608Metric, F.Cu at (-59.8, 256.2)
- added R39_R1: 1K, Resistor_SMD:R_0603_1608Metric, F.Cu at (-59.8, 258.7)
- added R4: 1K, Resistor_SMD:R_0603_1608Metric, F.Cu at (-67.8, 217.4)
- added R40_R1: 1K, Resistor_SMD:R_0603_1608Metric, F.Cu at (-59.8, 261.2)
- added R41_R1: 1K, Resistor_SMD:R_0603_1608Metric, F.Cu at (-59.8, 263.7)
- added R42_R1: 1K, Resistor_SMD:R_0603_1608Metric, F.Cu at (-59.8, 266.2)
- added R43_R1: 1K, Resistor_SMD:R_0603_1608Metric, F.Cu at (-59.8, 268.7)
- added R44_R1: 1K, Resistor_SMD:R_0603_1608Metric, F.Cu at (-59.8, 271.2)
- added R7: 1K, Resistor_SMD:R_0603_1608Metric, F.Cu at (-63.8, 199.8)
- added R706: 100R, Resistor_SMD:R_0603_1608Metric, F.Cu at (-55.8, 199.8)
- added R707: 10k, Resistor_SMD:R_0603_1608Metric, F.Cu at (-55.8, 202.4)
- added R708_R1: 100R, Resistor_SMD:R_0603_1608Metric, F.Cu at (-55.8, 253.7)
- added R709_R1: 10k, Resistor_SMD:R_0603_1608Metric, F.Cu at (-55.8, 256.2)
- added R710: 100R, Resistor_SMD:R_0603_1608Metric, F.Cu at (-55.8, 204.9)
- added R711: 100k, Resistor_SMD:R_0603_1608Metric, F.Cu at (-55.8, 207.4)
- added R712: 330R, Resistor_SMD:R_0603_1608Metric, F.Cu at (-55.8, 209.9)
- added R713_R1: 100R, Resistor_SMD:R_0603_1608Metric, F.Cu at (-55.8, 258.7)
- added R714_R1: 100k, Resistor_SMD:R_0603_1608Metric, F.Cu at (-55.8, 261.2)
- added R715_R1: 330R, Resistor_SMD:R_0603_1608Metric, F.Cu at (-55.8, 263.7)
- added R8: 1K, Resistor_SMD:R_0603_1608Metric, F.Cu at (-63.8, 202.4)
- added R9: 1K, Resistor_SMD:R_0603_1608Metric, F.Cu at (-63.8, 204.9)
- added RSW1: RSW1, Button_Switch_SMD:SW_SPST_SKQG_WithStem, F.Cu at (-24.5, 216.0)
- added RSW2_R1: RSW1, Button_Switch_SMD:SW_SPST_SKQG_WithStem, F.Cu at (-24.5, 269.8)
- added TP1: VBAT, TestPoint:TestPoint_Pad_D1.0mm, F.Cu at (-17.9, 197.4)
- added TP2: GND, TestPoint:TestPoint_Pad_D1.0mm, F.Cu at (-17.9, 200.4)
- added TP3: STS_LED_EN, TestPoint:TestPoint_Pad_D1.0mm, F.Cu at (-17.9, 203.5)
- added TP4_R1: VBAT_R, TestPoint:TestPoint_Pad_D1.0mm, F.Cu at (-17.9, 251.2)
- added TP5_R1: GND, TestPoint:TestPoint_Pad_D1.0mm, F.Cu at (-17.9, 254.3)
- added TP6_R1: STS_LED_EN_R, TestPoint:TestPoint_Pad_D1.0mm, F.Cu at (-17.9, 257.3)
- added U3: XIAO-nRF52840-Plus-SMD, Seeed_Studio_XIAO_Series:XIAO-nRF52840-Plus-SMD, B.Cu at (201.6, 111.9)
- added U5_R1: XIAO-nRF52840-Plus-SMD, Seeed_Studio_XIAO_Series:XIAO-nRF52840-Plus-SMD, B.Cu at (228.4, 111.9)
- SW1, SW10, SW11, SW12, SW13, SW14, SW15, SW16, SW17, SW18, SW19, SW2, SW20, SW21, SW22, SW23, SW24, SW25, SW26, SW27, SW28, SW29, SW3, SW30, SW31, SW32, SW33, SW34, SW35, SW36, SW37, SW38, SW39, SW4, SW40, SW5, SW6, SW7, SW8, SW9: footprint SW_MX_Choc_Hotswap -> willkeebs_keyboard:NF_LED_1206_SW_KS33_3_0_HS_1U
- turned SW1 to 180 degrees
- turned SW10 to 180 degrees
- turned SW11 to 180 degrees
- turned SW12 to 180 degrees
- turned SW13 to 180 degrees
- turned SW14 to 180 degrees
- turned SW15 to 180 degrees
- turned SW16 to 180 degrees
- turned SW17 to 180 degrees
- turned SW18 to 180 degrees
- turned SW19 to 165 degrees
- turned SW2 to 180 degrees
- turned SW20 to 151 degrees
- turned SW21 to 180 degrees
- turned SW22 to 180 degrees
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Connections:
- SW1 pad 1: outer_home_from -> Net-(D1-A)
- SW1 pad 2: outer_home_to -> COL0
- SW10 pad 1: middle_home_from -> Net-(D10-A)
- SW10 pad 2: middle_home_to -> COL3
- SW11 pad 1: middle_top_from -> Net-(D11-A)
- SW11 pad 2: middle_top_to -> COL3
- SW12 pad 1: index_bottom_from -> Net-(D12-A)
- SW12 pad 2: index_bottom_to -> COL4
- SW13 pad 1: index_home_from -> Net-(D13-A)
- SW13 pad 2: index_home_to -> COL4
- SW14 pad 1: index_top_from -> Net-(D14-A)
- SW14 pad 2: index_top_to -> COL4
- SW15 pad 1: inner_bottom_from -> Net-(D15-A)
- SW15 pad 2: inner_bottom_to -> COL5
- SW16 pad 1: inner_home_from -> Net-(D16-A)
- SW16 pad 2: inner_home_to -> COL5
- SW17 pad 1: inner_top_from -> Net-(D17-A)
- SW17 pad 2: inner_top_to -> COL5
- SW18 pad 1: inner_only_from -> Net-(D18-A)
- SW18 pad 2: inner_only_to -> COL3
- SW19 pad 1: home_only_from -> Net-(D19-A)
- SW19 pad 2: home_only_to -> COL4
- SW2 pad 1: outer_top_from -> Net-(D2-A)
- SW2 pad 2: outer_top_to -> COL0
- SW20 pad 1: outer_only_from -> Net-(D20-A)
- SW20 pad 2: outer_only_to -> COL5
- SW21 pad 1: mirror_outer_home_from -> Net-(D61_R1-A)
- SW21 pad 2: mirror_outer_home_to -> COL5_R
- SW22 pad 1: mirror_outer_top_from -> Net-(D62_R1-A)
- SW22 pad 2: mirror_outer_top_to -> COL5_R
- SW23 pad 1: mirror_pinky_bottom_from -> Net-(D63_R1-A)
- SW23 pad 2: mirror_pinky_bottom_to -> COL4_R
- SW24 pad 1: mirror_pinky_home_from -> Net-(D64_R1-A)
- SW24 pad 2: mirror_pinky_home_to -> COL4_R
- SW25 pad 1: mirror_pinky_top_from -> Net-(D72_R1-A)
- SW25 pad 2: mirror_pinky_top_to -> COL4_R
- SW26 pad 1: mirror_ring_bottom_from -> Net-(D73_R1-A)
- SW26 pad 2: mirror_ring_bottom_to -> COL3_R
- SW27 pad 1: mirror_ring_home_from -> Net-(D74_R1-A)
- SW27 pad 2: mirror_ring_home_to -> COL3_R
- SW28 pad 1: mirror_ring_top_from -> Net-(D75_R1-A)
- SW28 pad 2: mirror_ring_top_to -> COL3_R
- SW29 pad 1: mirror_middle_bottom_from -> Net-(D81_R1-A)
- SW29 pad 2: mirror_middle_bottom_to -> COL2_R
- SW3 pad 1: pinky_bottom_from -> Net-(D3-A)
- SW3 pad 2: pinky_bottom_to -> COL1
- SW30 pad 1: mirror_middle_home_from -> Net-(D82_R1-A)
- SW30 pad 2: mirror_middle_home_to -> COL2_R
- SW31 pad 1: mirror_middle_top_from -> Net-(D83_R1-A)
- SW31 pad 2: mirror_middle_top_to -> COL2_R
- SW32 pad 1: mirror_index_bottom_from -> Net-(D84_R1-A)
- SW32 pad 2: mirror_index_bottom_to -> COL1_R
- SW33 pad 1: mirror_index_home_from -> Net-(D85_R1-A)
- SW33 pad 2: mirror_index_home_to -> COL1_R
- SW34 pad 1: mirror_index_top_from -> Net-(D86_R1-A)
- SW34 pad 2: mirror_index_top_to -> COL1_R
- SW35 pad 1: mirror_inner_bottom_from -> Net-(D87_R1-A)
- SW35 pad 2: mirror_inner_bottom_to -> COL0_R
- SW36 pad 1: mirror_inner_home_from -> Net-(D88_R1-A)
- SW36 pad 2: mirror_inner_home_to -> COL0_R
- SW37 pad 1: mirror_inner_top_from -> Net-(D89_R1-A)
- SW37 pad 2: mirror_inner_top_to -> COL0_R
- SW38 pad 1: mirror_inner_only_from -> Net-(D90_R1-A)
- SW38 pad 2: mirror_inner_only_to -> COL0_R
- SW39 pad 1: mirror_home_only_from -> Net-(D91_R1-A)
- SW39 pad 2: mirror_home_only_to -> COL1_R
- SW4 pad 1: pinky_home_from -> Net-(D4-A)
- SW4 pad 2: pinky_home_to -> COL1
- SW40 pad 1: mirror_outer_only_from -> Net-(D92_R1-A)
- SW40 pad 2: mirror_outer_only_to -> COL2_R
- SW5 pad 1: pinky_top_from -> Net-(D5-A)
- SW5 pad 2: pinky_top_to -> COL1
- SW6 pad 1: ring_bottom_from -> Net-(D6-A)
- SW6 pad 2: ring_bottom_to -> COL2
- SW7 pad 1: ring_home_from -> Net-(D7-A)
- SW7 pad 2: ring_home_to -> COL2
- SW8 pad 1: ring_top_from -> Net-(D8-A)
- SW8 pad 2: ring_top_to -> COL2
- SW9 pad 1: middle_bottom_from -> Net-(D9-A)
- SW9 pad 2: middle_bottom_to -> COL3

Commit message: feat: added batteries and standoffs cutouts
Parts:
- removed J3, J4_R2: Conn_01x02, willkeebs_components:Pogo1x2-Right-Angle
- removed MH1, MH10_R1, MH2, MH3, MH4, MH5, MH5_R1, MH6_R1, MH7_R1, MH8_R1: MountingHole_2.2mm_M2, MountingHole:MountingHole_2.2mm_M2
- moved PSW1 0.28 mm to (187.0, 102.7)
Other:
- outline, holes or cut-outs redrawn
