File: keyboard/kicad/revisions/dormin-full/dormin.kicad_pcb (KiCad board)
At the start: 2 copper layers, 289.7 x 102.8 mm, 208 parts, among them J2 Conn_01x04, J6_R1 Conn_01x04, Q1 AO3400A, Q2 AO3407A, Q3_R1 AO3407A, Q4_R1 AO3400A, SW1 SW_Push, SW10 SW_Push, SW11 SW_Push, SW12 SW_Push, SW13 SW_Push, SW14 SW_Push, SW15 SW_Push, SW16 SW_Push, SW17 SW_Push, SW18 SW_Push, SW19 SW_Push, SW2 SW_Push, SW20 SW_Push, SW21 SW_Push, SW22 SW_Push, SW23 SW_Push, SW24 SW_Push, SW25 SW_Push, SW26 SW_Push, SW27 SW_Push, SW28 SW_Push, SW29 SW_Push, SW3 SW_Push, SW30 SW_Push, SW31 SW_Push, SW32 SW_Push, SW33 SW_Push, SW34 SW_Push, SW35 SW_Push, SW36 SW_Push, SW37 SW_Push, SW38 SW_Push, SW39 SW_Push, SW4 SW_Push, SW40 SW_Push, SW5 SW_Push, SW6 SW_Push, SW7 SW_Push, SW8 SW_Push, SW9 SW_Push, U1 Seeeduino Xiao nRF52840, U2 Seeeduino Xiao nRF52840

Commit message: feat: remove unused components for v1
Parts:
- removed U1, U2: Seeeduino Xiao nRF52840, Seeed_Studio_XIAO_Series:XIAO-nRF52840-SMD
- added D27: D_Schottky, Diode_SMD:D_SOD-523, F.Cu at (-39.7, 225.7)
- added D28: KPESD5V0S1UL, Diode_SMD:D_SOD-882, F.Cu at (-36.6, 225.7)
- added D47_R2: D_Schottky, Diode_SMD:D_SOD-523, F.Cu at (-39.7, 279.6)
- added D48_R2: KPESD5V0S1UL, Diode_SMD:D_SOD-882, F.Cu at (-36.6, 279.5)
- added F1: Polyfuse, Fuse:Fuse_1206_3216Metric, F.Cu at (-44.4, 226.2)
- added F2_R1: Polyfuse, Fuse:Fuse_1206_3216Metric, F.Cu at (-44.4, 280.0)
- added J1: Conn_01x06, willkeebs_misc:SMD_Conn_1x06_P2.54mm_Vertical, F.Cu at (-50.1, 200.9)
- added J3: Conn_01x02, willkeebs_components:Pogo1x2-Right-Angle, F.Cu at (-7.65, 230.4)
- added J4_R1: Conn_01x06, willkeebs_misc:SMD_Conn_1x06_P2.54mm_Vertical, F.Cu at (-50.1, 254.7)
- added J4_R2: Conn_01x02, willkeebs_components:Pogo1x2-Right-Angle, F.Cu at (-7.65, 238.5)
- added MH6: MountingHole_2.2mm_M2, MountingHole:MountingHole_2.2mm_M2, F.Cu at (-32.3, 221.5)
- added MH9_R1: MountingHole_2.2mm_M2, MountingHole:MountingHole_2.2mm_M2, F.Cu at (-32.3, 275.4)
- added U3: XIAO-nRF52840-Plus-SMD, Seeed_Studio_XIAO_Series:XIAO-nRF52840-Plus-SMD, B.Cu at (201.6, 111.9)
- added U5_R1: XIAO-nRF52840-Plus-SMD, Seeed_Studio_XIAO_Series:XIAO-nRF52840-Plus-SMD, B.Cu at (228.4, 111.9)
- JST2_R1, RSW1, RSW2_R1: moved to F.Cu
- moved JST2_R1 375.5 mm to (-65.8, 276.2), turned to 0 degrees
- moved RSW2_R1 327.4 mm to (-24.5, 269.8), turned to 0 degrees
- moved BT2_R1 322.4 mm to (-19.7, 263.2), turned to 0 degrees
- moved RSW1 173.3 mm to (-24.5, 216.0), turned to 0 degrees
Routing:
- net VBAT: track 12.9 -> 19.1 mm
